File: Commodore/Amiga/Amiga 1000/Amiga 1000.kicad_sch (KiCad schematic)
At the start: 51 parts, among them J10 DISK 0, J13 DISK 0 POWER, J7 DISK 1, J8 PARALLEL, J9 KBD, U6N MOS8520, U6P MOS8520, U7N- 7407, U7R- 7407

Commit message: More work on the Amiga 1000 schematic
I NEED A BREAK!
Parts:
- removed RN5: 1K, Resistor_THT:R_Array_SIP9, symbol Device:R_Network08_US
- added C10, C11, C12, C13, C14, C141, C15, C17, C18, C19, C7, C8, C9: .001, symbol Device:C_Small
- added C125: .1, symbol Device:C_Small
- added C126: 10µF, symbol Device:C_Polarized_Small
- added C16, C41, C42: .01, symbol Device:C_Small
- added D?: LED, symbol Device:LED
- added FB18, FB29, FB31, FB33, FB?: FERRITE_BEAD, symbol _RS_Commodore_Amiga_1000:FERRITE_BEAD
- added J15: CONN_LED, symbol _RS_Commodore_Amiga_1000:CONN_LED
- added J6: SERIAL, symbol _RS_Commodore_Amiga_1000:CONN_SERIAL
- added R30, R31, R38, R39, R40, R41, R42, R5, R6: 47, symbol Device:R_US
- added R49: 1K, symbol Device:R_US
- added R61: 560, symbol Device:R_US
- added R62: 1.2K, symbol Device:R_US
- added R99: 0.47, symbol Device:R_US
- added RN5, RN? (x7): 1K, symbol _RS_Commodore_Amiga_1000:RESISTOR_NET_10
- added U4A: MOS8362, Package_DIP:DIP-48_W15.24mm_LongPads, symbol _RS_Commodore_Amiga_1000:MOS8362
- added U4E: MOS8364, symbol _RS_Commodore_Amiga_1000:MOS8364
- added U4H-: 74F74, symbol _RS_Commodore_Amiga_1000:74F74
- added U6K, U6K-: LM1488, Package_DIP:DIP-14_W7.62mm_LongPads, symbol _RS_Commodore_Amiga_1000:LM1488
- added U6L-: LM1489A, Package_DIP:DIP-14_W7.62mm_LongPads, symbol _RS_Commodore_Amiga_1000:LM1489A
- added U7M-: 74LS04, symbol _RS_Commodore_Amiga_1000:74LS04
- added unit 4 of U7N-
- added unit 1 of U7N-
- added unit 6 of U7N-
- added U7P-: 7438, symbol _RS_Commodore_Amiga_1000:7438
- added unit 3 of U7R-
- J13: value DISK 0 POWER -> D0 PWR
Connections:
- net +12V: now also C16.1, J6.23 (+12V), R62.1
- net +5V: now also C125.1, C126.1, C42.1, FB31., J6.21 (+5V), R49.2, R99.1, R99.2, RN5.1, RN5.1, RN?.1, RN?.1, RN?.1, RN?.1, RN?.1, RN?.1, RN?.1, U4E.27 (VCC)
- net GND: now also C125.2, C126.2, J6.7 (GND), RN?.7, RN?.8, U4E.8 (GND)
- net GNDPWR: now also C10.2, C11.2, C12.2, C13.2, C14.2, C141.1, C15.2, C16.2, C17.2, C18.2, C19.2, C41.2, C42.2, C7.2, C8.2, C9.2, J15., J6.1 (GND)
- net ~{CHNG}: now also RN?.10
- net ~{DKRD}: now also RN5.3, U4E.37 (~{DKRD})
- net ~{DKWDB}: now also U7N-.2
- net ~{DKWD}: now also U4E.38 (~{DKWD}), U7N-.1
- net ~{DKWEB}: now also U7P-.8
- net ~{DRESB}: now also U7R-.6
- net ~{INDEX}: now also RN?.9
- net ~{MTR0D}: now also U7P-.6
- net ~{MTRXD}: now also U7P-.3
- net ~{MTR}: now also U7M-.9
- net ~{RDY}: now also RN5.2
- net ~{SEL0}: now also U7M-.11
- net ~{TKO}: now also RN?.5
- net ~{WPRO}: now also RN?.4
- net ~{RESET}: now reaches C22.2, J8.25 (~{RESET})
- net ~{RESET}: now also FB18., U7M-.6
- net ~{DSR}: now reaches U6N.5 (PA3)
- net ~{DSR}: now also R41.1, U6L-.1, U6L-.3
- net ~{CTS}: now reaches U6N.6 (PA4)
- net ~{CTS}: now also R40.1, U6L-.11, U6L-.13
- net ~{CD}: now reaches U6N.7 (PA5)
- net ~{CD}: now also R42.1, U6L-.4, U6L-.6
- net ~{RTS}: now reaches U6N.8 (PA6)
- net ~{RTS}: now also R39.1, U6K-.2, U6K-.3
- net ~{DTR}: now reaches U6N.9 (PA7)
- net ~{DTR}: now also U6K-.4, U6K-.5
- net ~{LED}: now reaches U6P.3 (PA1)
- net ~{LED}: now also U6K.10, U6K.9
- new net: U7M-.2, U7M-.3, U7M-.5
- new net: U7M-.4, U7N-.9
- new net: C18.1, J6.8 (CD), R42.2
- new net: C141.2, J15., R61.2, R62.2
- new net: C8.1, J6.15 (AUDOUT), R5.2
- new net: C7.1, J6.16 (AUDIN), R6.2
- new net: C15.1, FB29., J6.17 (EB)
- new net: C13.1, FB?., J6.18 (~{INT2})
- new net: C11.1, J6.2 (TXD), R38.2
- new net: C19.1, J6.20 (DTR), R31.2
- new net: C17.1, FB33., J6.25 (MRESB)
- new net: C10.1, J6.3 (RXD), R30.2
- new net: C9.1, J6.4 (RTS), R39.2
- new net: C14.1, J6.5 (CTS), R40.2
- new net: C12.1, J6.6 (DSR), R41.2
- new net: D?.1 (K), J15.1
- new net: D?.2 (A), J15.2
- new net: U4H-.9 (Q), U7P-.5
- new net: U4H-.11 (C), U7M-.10
- new net: U4H-.12 (D), U7M-.8, U7P-.2
- new net: U4E.11 (~{RES}), U7M-.1, U7P-.9
- new net: R61.1, U6K.8
- new net -5V: C41.1, J6.14 (-5V)
- new net CCK: U4E.28 (CCK)
- new net CCKQ: U4E.29 (CCKQ)
- new net D0: U4A.7 (D0), U4E.10 (D0)
- new net D1: U4A.6 (D1), U4E.9 (D1)
- new net D10: U4A.45 (D10), U4E.47 (D10)
- new net D11: U4A.44 (D11), U4E.46 (D11)
- new net D12: U4A.43 (D12), U4E.45 (D12)
- new net D13: U4A.42 (D13), U4E.44 (D13)
- new net D14: U4A.41 (D14), U4E.43 (D14)
- new net D15: U4A.40 (D15), U4E.42 (D15)
- new net D2: U4A.5 (D2), U4E.7 (D2)
- new net D3: U4A.4 (D3), U4E.6 (D3)
- new net D4: U4A.3 (D4), U4E.5 (D4)
- new net D5: U4A.2 (D5), U4E.4 (D5)
- new net D6: U4A.1 (D6), U4E.3 (D6)
- new net D7: U4A.48 (D7), U4E.2 (D7)
- new net D8: U4A.47 (D8), U4E.1 (D8)
- new net D9: U4A.46 (D9), U4E.48 (D9)
- new net DKWE: U4E.39 (DKWE), U7P-.10
- new net DTR: R31.1, U6K-.6
- new net EB: FB29.
- new net M0H: U4A.9 (M0H)
- new net M0V: U4A.38 (M0V)
- new net M1H: U4A.8 (M1H)
- new net M1V: U4A.39 (M1V)
- new net RGA1: U4A.10 (RGA8), U4E.26 (RGA1)
- new net RGA2: U4A.11 (RGA7), U4E.25 (RGA2)
- new net RGA3: U4A.12 (RGA6), U4E.24 (RGA3)
- new net RGA4: U4A.13 (RGA5), U4E.23 (RGA4)
- new net RGA5: U4A.14 (RGA4), U4E.22 (RGA5)
- new net RGA6: U4A.15 (RGA3), U4E.21 (RGA6)
- new net RGA7: U4A.16 (RGA2), U4E.20 (RGA7)
- new net RGA8: U4A.17 (RGA1), U4E.19 (RGA8)
- new net RXD: R30.1, U4E.41 (RXD), U6L-.10, U6L-.8
- new net TXD: R38.1, U4E.40 (TXD), U6K-.11, U6K-.12, U6K-.13
- new net ~{INT2}: FB?., U4E.16 (~{INT2})
- new net ~{INT3}: U4E.17 (~{INT3})
- new net ~{INT6}: U4E.18 (~{INT6})
- new net ~{IPL0}: U4E.13 (~{IPL0})
- new net ~{IPL1}: U4E.14 (~{IPL1})
- new net ~{IPL2}: U4E.15 (~{IPL2})
- new net ~{MCLK}: J6.24 (~{C2})
- new net ~{MRESB}: FB33., U7N-.12
- new net ~{RESB}: R49.1, U4H-.13 (~{R}), U7N-.13, U7N-.8, U7P-.1, U7P-.4, U7R-.5
- no-connect marks 1 -> 2
Other:
- note added: "3.58MHz"
- note added: "RN5 1K"
- moved on the sheet: C20, C21, C22, FB28, FB39, J13, J7
