File: Commodore/Amiga/Amiga 1000/Amiga 1000.kicad_sch (KiCad schematic)
At the start: 167 parts, among them J10 DISK 0, J11 RIGHT (1), J12 LEFT (0), J13 D0 PWR, J15 CONN_LED, J4 L, J5 R, J6 SERIAL, J7 DISK 1, J8 PARALLEL, J9 KBD, U4A MOS8362, U4E MOS8364, U4H- 74F74, U5G- LF347, U6K LM1488, U6K- LM1488, U6L- LM1489A, U6N MOS8520, U6P MOS8520, U7M- 74LS04, U7N- 7407, U7P- 7438, U7R- 7407

Commit message: Even more Amiga schematic work
Is it a problem if I'm seeing chips and wires in my DREAMS!??! :(
Parts:
- added C157, C178, C37, C38: .1, symbol Device:C_Small
- added C162, C163, C164, C165, C166, C169, C170, C171, C172, C173: .001, symbol Device:C_Small
- added C174: .01, symbol Device:C_Small
- added C175: 100 16V, symbol Device:C_Polarized_Small
- added FB34: FERRITE_BEAD, symbol _RS_Commodore_Amiga_1000:FERRITE_BEAD
- added J2: RF MOD, symbol _RS_Commodore_Amiga_1000:CONN_RF_MOD
- added Q18: 2SA733, Package_TO_SOT_THT:TO-92_Inline, symbol _RS_Commodore_Amiga_1000:2SA733
- added Q9: 2SB825, Package_TO_SOT_THT:TO-92_Inline, symbol _RS_Commodore_Amiga_1000:2SB825
- added R108: 200, symbol Device:R_US
- added R109, R136, R137, R138, R139: 470, symbol Device:R_US
- added R110: 1.5 .5W, symbol Device:R_US
- added R113: 39, symbol Device:R_US
- added R114, R115, R121, R122: 1, symbol Device:R_US
- added R116, R117, R118, R119, R123, R124, R125, R126: 220, symbol Device:R_US
- added R120, R127: 150, symbol Device:R_US
- added R141: 47, symbol Device:R_US
- added RN4, RN9: 100K, symbol _RS_Commodore_Amiga_1000:RESISTOR_NET_10
- added U1M: 74LS157, symbol _RS_Commodore_Amiga_1000:74LS157
- added unit 5 of U6K-
- gave numbers to parts that had none: 1
Connections:
- net +12V: now also U6K-.14 (V+)
- net +5V: now also C157.1, Q18.3 (E), R110.2, RN4.1, RN9.1, RN9.1, RN9.1, RN9.1, RN9.1, RN9.1, RN9.1, U1M.15 (E), U1M.16 (VCC)
- net -5V: now also U6K-.1 (V-)
- net GND: now also C157.2, U1M.8 (GND)
- net GNDPWR: now also J11.8 (SGND), J12.8 (SGND), C162.2, C163.2, C164.2, C165.2, C166.2, C169.2, C170.2, C171.2, C172.2, C173.2, C174.2, C175.1, C37.1, C38.1, J2.2 (SGND), J2.5 (SGND), R108.1
- net M0H: now also R137.1
- net M0V: now also R136.1
- net M1H: now also R139.1
- net M1V: now also R138.1
- net P0X: now also R122.1
- net P0Y: now also R121.1
- net P1X: now also R115.1
- net P1Y: now also R114.1
- net ~{FIR0}: now also R127.1
- net ~{FIR1}: now also R120.1
- net +5K: now reaches C36.1, FB19., J9.1 (+5V)
- net at J12.1 (FWRD_{0}): now also C173.1, R126.2
- net at J12.2 (BACK_{0}): now also C171.1, R125.2
- net at J12.3 (LEFT_{0}): now also C170.1, R124.2
- net at J12.4 (RIGHT_{0}): now also C169.1, R123.2
- net at J12.5 (POT_{0}X): now also R122.2
- net at J12.6 (~{FIRE_{0}}): now also C172.1, R127.2
- net +5LF: now reaches J12.7 (+5V)
- net +5LF: now also J11.7 (+5V), C174.1, C175.2, FB34.
- net at J12.9 (POT_{0}Y): now also R121.2
- net at R13.1: now also C37.2, J2.8 (R.AUD)
- net at R14.1: now also C38.2, J2.3 (L.AUD)
- net at J11.1 (FWRD_{1}): now also C166.1, R119.2
- net at J11.2 (BACK_{1}): now also C164.1, R118.2
- net at J11.3 (LEFT_{1}): now also C163.1, R117.2
- net at J11.4 (RIGHT_{1}): now also C162.1, R116.2
- net at J11.5 (POT_{1}X): now also R115.2
- net at J11.6 (~{FIRE_{1}}): now also C165.1, R120.2
- net at J11.9 (POT_{1}Y): now also R114.2
- new net: Q18.1 (B), R109.2, R113.1
- new net: R123.1, RN9.5, U1M.14 (A4)
- new net: Q9.1 (E), R110.1, R113.2
- new net: R126.1, RN9.2, U1M.3 (B1)
- new net: R117.1, RN9.9, U1M.11 (A3)
- new net: R119.1, RN9.8, U1M.10 (B3)
- new net: R137.2, U1M.12 (Y4)
- new net: R125.1, RN9.3, U1M.13 (B4)
- new net: R124.1, RN9.4, U1M.2 (A1)
- new net: R136.2, U1M.4 (Y1)
- new net: R116.1, RN4.7, U1M.5 (A2)
- new net: R118.1, RN9.6, U1M.6 (B2)
- new net: R139.2, U1M.7 (Y2)
- new net: R138.2, U1M.9 (Y3)
- new net: Q18.2 (C), Q9.3 (B), R108.2, R141.1
- new net: C178.1, R141.2
- new net +5L: C178.2, FB34., Q9.2 (C), R109.1
- new net C1: U1M.1 (S)
Other:
- note added: "= Shield = Digital = Video = Audio"
- note added: "SGND = DGND = VGND = AGND ="
- note removed: "+5K"
- moved on the sheet: C10, C11, C12, C13, C14, C15, C16, C17, C18, C19, C41, C42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

Commit message: You guessed it. Even more Amiga 1000 schematic work!
If I ever meet Michael Bowes, I'm gonna slap him with a wet noodle.
Parts:
- added C1, C117, C46, C52, C53, C86, C89: .1, symbol Device:C_Small
- added C118, C87: 10 10V, symbol Device:C_Polarized_Small
- added C176, C177: 470pF, symbol Device:C_Small
- added C2, C3, C4, C51, C55, C56, C57, C88, C90, C91: .01, symbol Device:C_Small
- added C45: 47pF, symbol Device:C_Small
- added C47: .001, symbol Device:C_Small
- added C48, C49, C50: 22 16V, symbol Device:C_Polarized_Small
- added C54: 100pF, symbol Device:C_Small
- added DL1: 400ns, symbol Device:DelayLine
- added FB35, FB36, FB37, FB38, FB40, FB42: FERRITE_BEAD, symbol _RS_Commodore_Amiga_1000:FERRITE_BEAD
- added J1: COMP, symbol Connector:Conn_Coaxial
- added J3: RGB, symbol _RS_Commodore_Amiga_1000:CONN_RGB
- added L1: 39µH, symbol Device:L_Small
- added Q1, Q2, Q?: 2SC2926, Package_TO_SOT_THT:TO-3PB-3_Vertical, symbol _RS_Commodore_Amiga_1000:2SC945A
- added Q10, Q4, Q5: 2SC945A, Package_TO_SOT_THT:TO-3PB-3_Vertical, symbol _RS_Commodore_Amiga_1000:2SC945A
- added Q8: 2SC752G, Package_TO_SOT_THT:TO-3PB-3_Vertical, symbol _RS_Commodore_Amiga_1000:2SC945A
- added R10, R12, R44: 220, symbol Device:R_US
- added R11, R16, R9: 75, symbol Device:R_US
- added R134, R17, R18, R19, R20, R21, R22: 47, symbol Device:R_US
- added R140: 220K, symbol Device:R_US
- added R142: 10K, symbol Device:R_US
- added R15: 470, symbol Device:R_US
- added R23, R24, R25: 75.0, symbol Device:R_US
- added R32, R33, R48: 3.3K, symbol Device:R_US
- added R35, R63: 3.92K, symbol Device:R_US
- added R37: 910, symbol Device:R_US
- added R43, R45, R47: 1K, symbol Device:R_US
- added R52: 1.69K, symbol Device:R_US
- added R53, R64, R68: 1000, symbol Device:R_US
- added R54, R65, R69: 2000, symbol Device:R_US
- added R55, R66, R70: 4020, symbol Device:R_US
- added R56, R67, R71: 8060, symbol Device:R_US
- added R57, R72, R76: 287, symbol Device:R_US
- added R58, R73, R77: 1150, symbol Device:R_US
- added R59, R74, R78: 100, symbol Device:R_US
- added R60, R75, R79: 49.9, symbol Device:R_US
- added T1: 166NNF-10264AG, symbol _RS_Commodore_Amiga_1000:TRANSFORMER-166NNF
- added U5A, U6A: 74HC244, symbol _RS_Commodore_Amiga_1000:74HC244
- added U7A: MC1377, Package_DIP:DIP-20_W7.62mm_LongPads, symbol _RS_Commodore_Amiga_1000:MC1377
Connections:
- net +12V: now also J2.7 (+12V), C1.2, C2.1, FB36., FB37., FB42., J3.22 (+12V), Q4.2 (C), Q5.2 (C), R33.2
- net +5V: now also U4A.19 (VCC), C117.2, C118.1, C3.1, C86.1, C87.1, C88.2, C89.2, C90.2, C91.2, FB35., J3.23 (+5V), Q1.2 (C), Q2.2 (C), Q?.2 (C), R142.1, R15.2, R58.2, R63.2, R73.2, R77.2, U5A.20 (VCC), U6A.20 (VCC)
- net -5V: now also C4.1, FB38., J3.21 (-5V)
- net Earth: now also U4A.37 (VSS), C1.1, C117.1, C118.2, C45.1, C46.2, C52.2, C53.2, C55.2, C56.2, C86.2, C87.2, C88.1, C89.1, C90.1, C91.1, DL1.3 (COMMUN), J3.16 (GND), J3.17 (GND), J3.18 (GND), J3.19 (GND), J3.20 (GND), Q8.3 (E), R140.1, R32.1, R43.1, R47.1, R57.1, R59.1, R72.1, R74.1, R76.1, R78.1, T1.3, U5A.1 (1OE), U5A.10 (GND), U5A.19 (2OE), U6A.1 (1OE), U6A.10 (GND), U6A.19 (2OE), U7A.15 (GND)
- net GND: now also J3.13 (GNDRTN), U7A.20 (N/P)
- net GNDPWR: now also C176.1, C177.1, C2.2, C3.2, C4.2, J1.2 (Ext), Q10.3 (E), R10.1, R12.1
- net at J2.4 (VIDEO): now also C177.2, R11.2
- net at U4A.18 (~{BURST}): now also U6A.2 (1A0)
- net at U4A.20 (R0): now also U5A.4 (1A1)
- net at U4A.21 (R1): now also U5A.6 (1A2)
- net at U4A.22 (R2): now also U5A.2 (1A0)
- net at U4A.23 (R3): now also U5A.8 (1A3)
- net at U4A.24 (B0): now also U5A.17 (2A0)
- net at U4A.25 (B1): now also U5A.15 (2A1)
- net at U4A.26 (B2): now also U5A.13 (2A2)
- net at U4A.27 (B3): now also U5A.11 (2A3)
- net at U4A.28 (G0): now also U6A.17 (2A0)
- net at U4A.29 (G1): now also U6A.15 (2A1)
- net at U4A.30 (G2): now also U6A.13 (2A2)
- net at U4A.31 (G3): now also U6A.11 (2A3)
- net at U4A.33 (~{ZD}): now also U6A.4 (1A1)
- new net: Q1.1 (B), R64.2, R65.2, R66.2, R67.2, R72.2, R73.1
- new net: R35.1, U7A.1 (T_{r})
- new net: R35.2, R52.2, R63.1
- new net: C48.2, R74.2, R75.1
- new net: Q1.3 (E), R25.1, R75.2
- new net: C176.2, J1.1 (In), R9.2
- new net: Q?.1 (B), R68.2, R69.2, R70.2, R71.2, R76.2, R77.1
- new net: Q?.3 (E), R23.1, R79.2
- new net: DL1.1, R43.2, U7A.8 (-Y_{in})
- new net: DL1.2, R45.2
- new net: J3.8 (G_{#}), R18.2
- new net: C49.1, U7A.5 (B)
- new net: C49.2, R78.2, R79.1
- new net: C53.1, U7A.12 (R-Y_{clamp})
- new net: Q2.3 (E), R24.1, R60.2
- new net: C51.1, R37.2
- new net: C51.2, L1.2
- new net: J3.10 (~{CS}), R16.2
- new net: J3.11 (~{HS}), R142.2, R21.2
- new net: J3.12 (~{VS}), R22.2
- new net: J3.14 (~{ZD}), R134.2
- new net: FB40., J3.15 (~{C1})
- new net: J3.6 (I), R20.2
- new net: J3.7 (R_{#}), R19.2
- new net: J3.9 (B_{#}), R17.2
- new net: Q10.1 (B), Q8.2 (C), R33.1
- new net: Q4.1 (B), Q5.1 (B), U7A.9 (CV_{out})
- new net: Q4.3 (E), R10.2, R9.1
- new net: C45.2, C47.1, R32.2, T1.1
- new net: Q5.3 (E), R11.1, R12.2
- new net: C47.2, U7A.10 (CHROMA_{in})
- new net: C52.1, U7A.11 (B-Y_{clamp})
- new net: R44.1, U7A.13 (CHROMA_{out})
- new net: C46.1, FB36., T1.4, U7A.14 (V+)
- new net: C57.2, U7A.17 (OSC_{in})
- new net: C56.1, R140.2, U7A.19 (ɸ_{m})
- new net: C48.1, U7A.3 (R)
- new net: C50.1, U7A.4 (G)
- new net: R45.1, U7A.6 (-Y_{out})
- new net: C55.1, U7A.7 (V_{clamp})
- new net: Q2.1 (B), R53.2, R54.2, R55.2, R56.2, R57.2, R58.1
- new net: C57.1, R47.2, R48.2
- new net: C54.1, T1.5
- new net: C54.2, R44.2
- new net: C50.2, R59.2, R60.1
- new net: L1.1, R48.1
- new net: Q10.2 (C), R15.1, R16.1
- new net B: J3.5 (B_{∩}), R23.2
- new net BB0: R20.1, R71.1, U5A.3 (2Y0)
- new net BB1: R70.1, U5A.5 (2Y1)
- new net BB2: R69.1, U5A.7 (2Y2)
- new net BB3: R19.1, R68.1, U5A.9 (2Y3)
- new net BG0: R56.1, U6A.3 (2Y0)
- new net BG1: R55.1, U6A.5 (2Y1)
- new net BG2: R54.1, U6A.7 (2Y2)
- new net BG3: R18.1, R53.1, U6A.9 (2Y3)
- new net BR0: R67.1, U5A.16 (1Y1)
- new net BR1: R66.1, U5A.14 (1Y2)
- new net BR2: R65.1, U5A.18 (1Y0)
- new net BR3: R17.1, R64.1, U5A.12 (1Y3)
- new net G: J3.4 (G_{∩}), R24.2
- new net R: J3.3 (R_{∩}), R25.2
- new net ~{BBST}: R52.1, U6A.18 (1Y0)
- new net ~{BHS}: R134.1, U6A.16 (1Y1)
- new net ~{C1U}: FB40.
- new net ~{C4U}: R37.1
- new net ~{CSY}: U6A.6 (1A2)
- new net ~{C}: Q8.1 (B), U6A.12 (1Y3), U7A.2 (~{SYNC})
- new net ~{HSY}: R21.1
- new net ~{VSY}: R22.1
- new net ~{XCLKEN}: J3.2 (~{XCLKEN})
- new net ~{XCLK}: J3.1 (~{XCLK})
- no-connect marks 2 -> 6
Other:
- note added: "0.47 x4"
- moved on the sheet: C37, C38, J2, U4A

Commit message: Surprise!  More Amiga 1000 schematic work!
I need a break..................
Parts:
- added C123: .1, symbol Device:C_Small
- added C124: 10 10V, symbol Device:C_Polarized_Small
- added R111, R112: 1K, symbol Device:R_US
- added RN1: 1K, symbol _RS_Commodore_Amiga_1000:RESISTOR_NET_10
- added U1J: 74F399, symbol _RS_Commodore_Amiga_1000:74F399
- added U2H: 74F374, symbol _RS_Commodore_Amiga_1000:74F374
- added U4C: MOS8361, symbol _RS_Commodore_Amiga_1000:MOS8361
- added unit 1 of U4H-
- added U4J: 74LS244, symbol _RS_Commodore_Amiga_1000:74LS244_U4J_MAINBOARD
- gave numbers to parts that had none: 1
Connections:
- net +5V: now also C123.2, C124.2, R111.2, R112.2, RN1.1, RN1.1, RN1.1, RN1.1, RN1.1, RN1.1, RN1.1, RN1.1, RN1.1, U4C.10 (VCC)
- net CCK: now also U4A.36 (~{CAS}), U4C.25 (CCK)
- net CCKQ: now also U4C.26 (CCKQ)
- net D0: now also U4C.9 (D0)
- net D1: now also U4C.8 (D1)
- net D10: now also U4C.47 (D10)
- net D11: now also U4C.46 (D11)
- net D12: now also U4C.45 (D12)
- net D13: now also U4C.44 (D13)
- net D14: now also U4C.43 (D14)
- net D15: now also U4C.42 (D15)
- net D2: now also U4C.7 (D2)
- net D3: now also U4C.6 (D3)
- net D4: now also U4C.5 (D4)
- net D5: now also U4C.4 (D5)
- net D6: now also U4C.3 (D6)
- net D7: now also U4C.2 (D7)
- net D8: now also U4C.1 (D8)
- net D9: now also U4C.48 (D9)
- net GND: now also C123.1, C124.1, U4C.27 (GND), U4C.41 (GND)
- net RGA1: now also RN1.10, U4C.24 (RGA1), U4J.12 (O3a)
- net RGA2: now also RN1.9, U4C.23 (RGA2), U4J.9 (O0b)
- net RGA3: now also RN1.8, U4C.22 (RGA3), U4J.14 (O2a)
- net RGA4: now also RN1.7, U4C.21 (RGA4), U4J.7 (O1b)
- net RGA5: now also RN1.6, U4C.20 (RGA5), U4J.16 (O1a)
- net RGA6: now also RN1.5, U4C.19 (RGA6), U4J.5 (O2b)
- net RGA7: now also RN1.4, U4C.18 (RGA7), U4J.18 (O0a)
- net RGA8: now also RN1.3, U4C.17 (RGA8), U4J.3 (O3b)
- net ~{CSY}: now also U6A.8 (1A3), U4C.39 (~{CSY}); no longer U6A.6 (1A2)
- net ~{FIR0}: now also U4C.37 (~{LP})
- net ~{HSY}: now also U6A.6 (1A2), U4C.40 (~{HSY})
- net ~{INT3}: now also U4C.12 (~{INT3})
- net ~{VSY}: now also U4C.38 (~{VSY})
- net PU: now reaches U4H-.10 (~{S})
- net PU: now also R111.1, U1J.11 (I0c), U1J.12 (I1c), U1J.13 (I1d), U1J.14 (I0d), U4H-.4 (~{S})
- net ~{RES}: now reaches U4E.11 (~{RES}), U7M-.1, U7P-.9
- net ~{RES}: now also U4C.11 (~{RES})
- net DMAL: now reaches U4E.12 (DMAL)
- net DMAL: now also U4C.13 (DMAL)
- new net: R112.1, U4H-.1 (~{R})
- new net: U2H.8 (D0), U4C.28 (DRA0)
- new net: U2H.7 (D1), U4C.29 (DRA1)
- new net: U2H.4 (D2), U4C.30 (DRA2)
- new net: U2H.3 (D3), U4C.31 (DRA3)
- new net: U2H.18 (D4), U4C.32 (DRA4)
- new net: U2H.17 (D5), U4C.33 (DRA5)
- new net: U2H.14 (D6), U4C.34 (DRA6)
- new net: U2H.13 (D7), U4C.35 (DRA7)
- new net: U1J.4 (I1a), U4C.36 (DRA8), U4H-.2 (D)
- new net: U1J.5 (I1b), U4H-.5 (Q)
- new net A1: U4J.8 (I3a)
- new net A17: U1J.3 (I0a)
- new net A18: U1J.6 (I0b)
- new net A2: U4J.11 (I0b)
- new net A3: U4J.6 (I2a)
- new net A4: U4J.13 (I1b)
- new net A5: U4J.4 (I1a)
- new net A6: U4J.15 (I2b)
- new net A7: U4J.2 (I0a)
- new net A8: U4J.17 (I3b)
- new net C4: U1J.9 (CP)
- new net DAC: U2H.11 (Cp), U4H-.3 (C)
- new net MA17: U1J.7 (Qb)
- new net MA18: U1J.2 (Qa)
- new net RA0: U2H.9 (Q0)
- new net RA1: U2H.6 (Q1)
- new net RA2: U2H.5 (Q2)
- new net RA3: U2H.2 (Q3)
- new net RA4: U2H.19 (Q4)
- new net RA5: U2H.16 (Q5)
- new net RA6: U2H.15 (Q6)
- new net RA7: U2H.12 (Q7)
- new net ~{ARW}: U4C.16 (~{ARW})
- new net ~{BLS}: U4C.14 (~{BLS})
- new net ~{DAE}: U2H.1 (OE)
- new net ~{DBR}: U4C.15 (~{DBR})
- new net ~{RE}: U1J.1 (S)
- new net ~{RGAE}: U4J.1 (OEa), U4J.19 (OEb)
- no-connect marks 6 -> 11
Other:
- note added: "AGNUS"
- note added: "RN1 1K"
- moved on the sheet: C1, C10, C11, C12, C13, C14, C15, C157, C16, C162, C163, C164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

Commit message: minor changes
Other:
- note removed: "AGNUS"
- note removed: "CIA"
- note removed: "DENISE"
- note removed: "PAULA"
Changed lines of the file:
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@@
     (stroke (width 0) (type default) (color 0 0 0 0))
   )
-  (bus_entry (at 220.98 236.22) (size 2.54 2.54)
+  (bus_entry (at 220.98 314.96) (size 2.54 2.54)
     (stroke (width 0) (type default) (color 0 0 0 0))
   )
-  (bus_entry (at 220.98 238.76) (size 2.54 2.54)
+  (bus_entry (at 220.98 320.04) (size 2.54 2.54)
     (stroke (width 0) (type default) (color 0 0 0 0))
   )
@@
     (stroke (width 0) (type default) (color 0 0 0 0))
   )
-  (wire (pts (xy 241.3 317.5) (xy 241.3 238.76))
-    (stroke (width 0) (type default) (color 0 0 0 0))
-  )
   (wire (pts (xy 386.08 48.26) (xy 386.08 50.8))
     (stroke (width 0) (type default) (color 0 0 0 0))
@@
     (stroke (width 0) (type default) (color 0 0 0 0))
   )
-  (wire (pts (xy 317.5 322.58) (xy 240.03 322.58))
-    (stroke (width 0) (type default) (color 0 0 0 0))
-  )
   (wire (pts (xy 365.76 386.08) (xy 369.57 386.08))
     (stroke (width 0) (type default) (color 0 0 0 0))
@@
     (stroke (width 0) (type default) (color 0 0 0 0))
   )
-  (bus (pts (xy 220.98 236.22) (xy 220.98 238.76))
+  (bus (pts (xy 220.98 314.96) (xy 220.98 320.04))
     (stroke (width 0) (type default) (color 0 0 0 0))
   )
@@
     (stroke (width 0) (type default) (color 0 0 0 0))
   )
-  (wire (pts (xy 240.03 322.58) (xy 240.03 241.3))
-    (stroke (width 0) (type default) (color 0 0 0 0))
-  )
   (wire (pts (xy 170.18 69.85) (xy 170.18 52.07))
     (stroke (width 0) (type default) (color 0 0 0 0))
@@
     (stroke (width 0) (type default) (color 0 0 0 0))
   )
-  (wire (pts (xy 317.5 317.5) (xy 241.3 317.5))
-    (stroke (width 0) (type default) (color 0 0 0 0))
-  )
   (bus (pts (xy 406.4 63.5) (xy 421.64 63.5))
     (stroke (width 0) (type default) (color 0 0 0 0))
@@
     (stroke (width 0) (type default) (color 0 0 0 0))
   )
-  (bus (pts (xy 220.98 228.6) (xy 220.98 236.22))
+  (bus (pts (xy 220.98 228.6) (xy 220.98 314.96))
     (stroke (width 0) (type default) (color 0 0 0 0))
   )
@@
     (stroke (width 0) (type default) (color 0 0 0 0))
   )
-  (wire (pts (xy 223.52 238.76) (xy 241.3 238.76))
+  (wire (pts (xy 223.52 317.5) (xy 317.5 317.5))
     (stroke (width 0) (type default) (color 0 0 0 0))
   )
@@
     (stroke (width 0) (type default) (color 0 0 0 0))
   )
-  (wire (pts (xy 223.52 241.3) (xy 240.03 241.3))
+  (wire (pts (xy 223.52 322.58) (xy 317.5 322.58))
     (stroke (width 0) (type default) (color 0 0 0 0))
   )
@@
     (effects (font (size 1.27 1.27)) (justify left bottom))
   )
-  (text "DENISE" (at 478.79 434.34 90)
-    (effects (font (size 2.54 2.54)) (justify left bottom))
-  )
   (text "= Shield\n= Digital\n= Video\n= Audio" (at 571.5 171.45 0)
     (effects (font (size 2.54 2.54)) (justify left bottom))
@@
     (effects (font (size 2.54 2.54)) (justify left bottom))
   )
-  (text "CIA" (at 250.19 132.08 0)
-    (effects (font (size 2.54 2.54)) (justify left bottom))
-  )
-  (text "CIA" (at 151.13 132.08 0)
-    (effects (font (size 2.54 2.54)) (justify left bottom))
-  )
-  (text "AGNUS" (at 254 394.97 90)
-    (effects (font (size 2.54 2.54)) (justify left bottom))
-  )
   (text "RN5\n1K" (at 265.43 62.23 0)
     (effects (font (size 1.27 1.27)) (justify left bottom))
   )
-  (text "PAULA" (at 478.79 212.09 90)
-    (effects (font (size 2.54 2.54)) (justify left bottom))
-  )
   (text "3.58MHz" (at 1037.59 227.33 0)
     (effects (font (size 1.27 1.27)) (justify left bottom))
@@
     (effects (font (size 1.27 1.27)) (justify right bottom))
   )
-  (label "A18" (at 238.76 241.3 180)
+  (label "A18" (at 238.76 322.58 180)
     (effects (font (size 1.27 1.27)) (justify right bottom))
   )
@@
     (effects (font (size 1.27 1.27)) (justify left bottom))
   )
-  (label "A18" (at 318.77 322.58 180)
+  (label "A18" (at 317.5 322.58 180)
     (effects (font (size 1.27 1.27)) (justify right bottom))
   )
@@
     (effects (font (size 1.27 1.27)) (justify left bottom))
   )
-  (label "A17" (at 238.76 238.76 180)
+  (label "A17" (at 238.76 317.5 180)
     (effects (font (size 1.27 1.27)) (justify right bottom))
   )
@@
     (effects (font (size 1.27 1.27)) (justify right bottom))
   )
-  (label "A17" (at 318.77 317.5 180)
+  (label "A17" (at 317.5 317.5 180)
     (effects (font (size 1.27 1.27)) (justify right bottom))
   )
@@
     (pin "3")
   )
-  (symbol (lib_id "_RS_Commodore_Amiga_1000:MOS8520") (at 248.92 137.16 90) (unit 1)
+  (symbol (lib_name "MOS8520_1") (lib_id "_RS_Commodore_Amiga_1000:MOS8520") (at 248.92 137.16 90) (unit 1)
     (in_bom yes) (on_board yes)
-    (property "Reference" "U6N" (id 0) (at 292.1 129.54 90)
+    (property "Reference" "U6N" (id 0) (at 312.42 129.54 90)
       (effects (font (size 1.27 1.27)) (justify left))
     )
-    (property "Value" "MOS8520" (id 1) (at 280.67 129.54 90)
+    (property "Value" "MOS8520" (id 1) (at 261.62 129.54 90)
       (effects (font (size 1.27 1.27)) (justify left))
     )
@@
   (symbol (lib_id "_RS_Commodore_Amiga_1000:MOS8520") (at 149.86 137.16 90) (unit 1)
     (in_bom yes) (on_board yes)
-    (property "Reference" "U6P" (id 0) (at 193.04 129.54 90)
+    (property "Reference" "U6P" (id 0) (at 213.36 129.54 90)
       (effects (font (size 1.27 1.27)) (justify left))
     )
-    (property "Value" "MOS8520" (id 1) (at 181.61 129.54 90)
+    (property "Value" "MOS8520" (id 1) (at 162.56 129.54 90)
       (effects (font (size 1.27 1.27)) (justify left))
     )
