File: Commodore/Amiga/Amiga 1000/Amiga 1000.kicad_sch (KiCad schematic)
At the start: 316 parts, among them J1 COMP, J10 DISK 0, J11 RIGHT (1), J12 LEFT (0), J13 D0 PWR, J15 CONN_LED, J2 RF MOD, J3 RGB, J4 L, J5 R, J6 SERIAL, J7 DISK 1, J8 PARALLEL, J9 KBD, Q1 2SC2926, Q10 2SC945A, Q18 2SA733, Q2 2SC2926, Q4 2SC945A, Q5 2SC945A, Q8 2SC752G, Q9 2SB825, T1 166NNF-10264AG, U1J 74F399, U1M 74LS157, U2H 74F374, U4A MOS8362, U4C MOS8361, U4E MOS8364, U4H- 74F74, U4J 74LS244, U5A 74HC244, U5G- LF347, U6A 74HC244, U6K LM1488, U6K- LM1488, U6L- LM1489A, U6N MOS8520, U6P MOS8520, U7A MC1377, U7M- 74LS04, U7N- 7407, U7P- 7438, U7R- 7407

Commit message: Even. More. Amiga 1000. Schematic. Work.
I'm inching ever closer!!!!
Parts:
- added C114, C134, C135: 10 10V, symbol Device:C_Polarized_Small
- added C116: .1, symbol Device:C_Small
- added C133: 0.1, symbol Device:C_Small
- added C139, C140: .01, symbol Device:C_Small
- added CR2: 1N4148, symbol Device:D
- added P1: CONN_EXPANSION, symbol _RS_Commodore_Amiga_1000:CONN_EXPANSION
- added R100, R103, R104: 1K, symbol Device:R_US
- added R101: 1M, symbol Device:R_US
- added R102: 10K, symbol Device:R_US
- added R105: 100K 10%, symbol Device:R_US
- added R106: 22K 10%, symbol Device:R_US
- added RN-, RN6-: 10K, symbol _RS_Commodore_Amiga_1000:RESISTOR_NET_10
- added RN7-, RN7-? (x3): 1K, symbol _RS_Commodore_Amiga_1000:RESISTOR_NET_10
- added RN8-, RN8-? (x4): 2.7K, symbol _RS_Commodore_Amiga_1000:RESISTOR_NET_10
- added TP1: TestPoint, symbol Connector:TestPoint
- added U4M-: LM2901, symbol _RS_Commodore_Amiga_1000:LM2901
- added U5L: PALEN - U5L, symbol _RS_Commodore_Amiga_1000:PALEN - U5L
- added U5M: PALCAS - U5M, symbol _RS_Commodore_Amiga_1000:PALCAS - U5M
- added U5N, U5P: 23256, Package_DIP:DIP-28_W15.24mm_LongPads, symbol _RS_Commodore_Amiga_1000:TMM2356P
- added U6M-: 74LS32, symbol _RS_Commodore_Amiga_1000:74LS32
- added U6S: Motorola_68000, Package_DIP:DIP-64_W15.24mm, symbol _RS_Commodore_Amiga_1000:Motorola_68000
- added U7F-: 74LS04, symbol _RS_Commodore_Amiga_1000:74LS04
- added unit 4 of U7P-
- added W1, W2, W3, W4, W5: UNKNOWN_W_SYMBOL, symbol _RS_Commodore_Amiga_1000:UNKNOWN_W_SYMBOL
Connections:
- net ~{RGAE} is gone; now on net DMAL: U4J.1 (OEa), U4J.19 (OEb)
- net +12V: now also C139.2, P1.10 (+12)
- net +5V: now also RN1., RN1., RN1., RN1., RN1., RN1., RN1., RN1., RN1., RN4., RN5., RN5., RN5., RN5., RN5., RN5., RN5., RN5., RN5., RN9., RN9., RN9., RN9., RN9., RN9., RN9., U6N.20 (VCC), U6P.20 (VCC), C114.1, C116.2, CR2.1 (K), P1.5 (+5V), P1.6 (+5V), R100.2, R103.2, R105.2, R106.2, RN-., RN6-., RN6-., RN6-., RN6-., RN6-., RN6-., RN7-., RN7-., RN7-., RN7-., RN7-., RN7-., RN7-?., RN7-?., RN7-?., RN8-., RN8-?., RN8-?., RN8-?., RN8-?., U4M-.3 (V+), U6S.14 (VCC), U6S.49 (VCC), W2.; no longer RN1.1, RN1.1, RN1.1, RN1.1, RN1.1, RN1.1, RN1.1, RN1.1, RN1.1, RN4.1, RN5.1, RN5.1, RN5.1, RN5.1, RN5.1, RN5.1, RN5.1, RN5.1, RN5.1, RN9.1, RN9.1, RN9.1, RN9.1, RN9.1, RN9.1, RN9.1
- net -5V: now also C140.2, P1.8 (-5V)
- net A1: now also P1.29 (A1), U5N.10 (A1), U5P.10 (A1), U6S.29 (A1)
- net A17: now also P1.47 (A17), U6S.45 (A17), W4.
- net A18: now also P1.52 (A18), U6S.46 (A18)
- net A2: now also P1.27 (A2), U5N.9 (A2), U5P.9 (A2), U6S.30 (A2)
- net A3: now also P1.26 (A3), U5N.8 (A3), U5P.8 (A3), U6S.31 (A3)
- net A4: now also P1.24 (A4), U5N.7 (A4), U5P.7 (A4), U6S.32 (A4)
- net A5: now also P1.21 (A5), U5N.6 (A5), U5P.6 (A5), U6S.33 (A5)
- net A6: now also P1.23 (A6), U5N.5 (A6), U5P.5 (A6), U6S.34 (A6)
- net A7: now also P1.28 (A7), U5N.4 (A7), U5P.4 (A7), U6S.35 (A7)
- net A8: now also U6N.38 (A0), U6P.38 (A0), P1.30 (A8), U5N.3 (A8), U5P.3 (A8), U6S.36 (A8)
- net EB: now also U6M-.11
- net GND: now also U6N.1 (GND), U6P.1 (GND), C114.2, C116.1, C133.1, C133.2, C134.2, C135.2, C139.1, C140.1, P1.1 (DGND), P1.12 (~{CONFIG}), P1.13 (DGND), P1.2 (DGND), P1.25 (DGND), P1.3 (DGND), P1.37 (DGND), P1.4 (DGND), P1.49 (DGND), P1.61 (DGND), P1.73 (DGND), P1.85 (DGND), R102.1, R103.1, R104.1, R104.2, U4M-.12 (V-), U4M-.5 (+), U4M-.7 (+), U4M-.9 (+), U6M-.13, U6M-.5, U6S.16 (GND), U6S.53 (GND), W3.
- net KCLK: now also U4M-.6 (-)
- net ~{BHS}: now also U6N.19 (TOD)
- net ~{INT2}: now also P1.19 (~{INT2}), RN8-.7
- net ~{INT6}: now also P1.22 (~{INT6}), RN8-?.6
- net ~{IPL0}: now also P1.40 (~{IPL_{0}}), RN8-?.8, U6S.25 (~{IPL_{0}})
- net ~{IPL1}: now also P1.42 (~{IPL_{1}}), RN8-?.9, U6S.24 (~{IPL_{1}})
- net ~{IPL2}: now also P1.44 (~{IPL_{2}}), RN8-?.10, U6S.23 (~{IPL_{2}})
- net ~{RES}: now also U6N.34 (~{RES}), U6P.34 (~{RES}), P1.53 (~{RES}), RN6-.7, U4M-.14, U6S.18 (~{RESET})
- net ~{PRWD}: now reaches U6N.22 (R/~{W})
- net ~{PRWD}: now also U6P.22 (R/~{W}), U6M-.6
- net at U6N.23 (~{CS}): now also U6M-.8
- net E: now reaches U6N.25 (ɸ2)
- net E: now also U6P.25 (ɸ2), P1.50 (E), U6M-.12, U6S.20 (E)
- net PD15: now reaches U6N.26 (D7)
- net PD15: now also P1.63 (PD15), U5N.19 (D7), U6S.54 (D15)
- net PD14: now reaches U6N.27 (D6)
- net PD14: now also P1.65 (PD14), U5N.18 (D6), U6S.55 (D14)
- net PD13: now reaches U6N.28 (D5)
- net PD13: now also P1.67 (PD13), U5N.17 (D5), U6S.56 (D13)
- net PD12: now reaches U6N.29 (D4)
- net PD12: now also P1.69 (PD12), U5N.16 (D4), U6S.57 (D12)
- net PD11: now reaches U6N.30 (D3)
- net PD11: now also P1.71 (PD11), U5N.15 (D3), U6S.58 (D11)
- net PD10: now reaches U6N.31 (D2)
- net PD10: now also P1.76 (PD10), U5N.13 (D2), U6S.59 (D10)
- net PD9: now reaches U6N.32 (D1)
- net PD9: now also P1.78 (PD9), U5N.12 (D1), U6S.60 (D9)
- net PD8: now reaches U6N.33 (D0)
- net PD8: now also P1.80 (PD8), U5N.11 (D0), U6S.61 (D8)
- net A11: now reaches U6N.35 (A3)
- net A11: now also U6P.35 (A3), P1.36 (A11), U5N.21 (A11), U5P.21 (A11), U6S.39 (A11)
- net A10: now reaches U6N.36 (A2)
- net A10: now also U6P.36 (A2), P1.34 (A10), U5N.24 (A10), U5P.24 (A10), U6S.38 (A10)
- net A9: now reaches U6N.37 (A1)
- net A9: now also U6P.37 (A1), P1.32 (A9), U5N.25 (A9), U5P.25 (A9), U6S.37 (A9)
- net TICK: now reaches U6P.19 (TOD)
- net OVL: now reaches U6P.2 (PA0)
- net OVL: now also U5L.6 (I6)
- net at U6P.23 (~{CS}): now also U6M-.3
- net PD7: now reaches U6P.26 (D7)
- net PD7: now also P1.82 (PD7), U5P.19 (D7), U6S.62 (D7)
- net PD6: now reaches U6P.27 (D6)
- net PD6: now also P1.84 (PD6), U5P.18 (D6), U6S.63 (D6)
- net PD5: now reaches U6P.28 (D5)
- net PD5: now also P1.86 (PD5), U5P.17 (D5), U6S.64 (D5)
- net PD4: now reaches U6P.29 (D4)
- net PD4: now also P1.83 (PD4), U5P.16 (D4), U6S.1 (D4)
- net PD3: now reaches U6P.30 (D3)
- net PD3: now also P1.81 (PD3), U5P.15 (D3), U6S.2 (D3)
- net PD2: now reaches U6P.31 (D2)
- net PD2: now also U5P.13 (D2), U6S.3 (D2)
- net PD1: now reaches U6P.32 (D1)
- net PD1: now also P1.77 (PD1), U5P.12 (D1), U6S.4 (D1)
- net PD0: now reaches U6P.33 (D0)
- net PD0: now also P1.75 (PD0), U5P.11 (D0), U6S.5 (D0)
- new net: C134.1, CR2.2 (A), R105.1, TP1.1, U4M-.10 (-), U4M-.2
- new net: U5N.26 (A14), U5P.26 (A14), W3.
- new net: C135.1, R106.1, U4M-.1, U4M-.4 (-)
- new net: U5N.20 (~{CE}), U5P.20 (~{CE}), W5.
- new net: U5N.20 (~{CE}), U5P.20 (~{CE}), U7F-.13, W4., W5.
- new net: U7F-.12, W5.
- new net: U5N.1 (?), U5P.1 (?)
- new net: U5N.22 (~{OE}), U5P.22 (~{OE})
- new net: U5N.27 (A15), U5P.27 (A15), W1., W2.
- new net: R101.1, R102.2, U4M-.11 (+)
- new net: R100.1, R101.2, U4M-.13, U4M-.8 (-), U7P-.12, U7P-.13
- new net A12: P1.38 (A12), U5N.23 (A12), U5P.23 (A12), U6M-.1, U6S.40 (A12)
- new net A13: P1.39 (A13), U5N.2 (A13), U5P.2 (A13), U6M-.9, U6S.41 (A13)
- new net A14: P1.41 (A14), U5N.26 (A14), U5P.26 (A14), U6S.42 (A14), W3.
- new net A15: P1.43 (A15), U5N.27 (A15), U5P.27 (A15), U6S.43 (A15), W1.
- new net A16: P1.45 (A16), U6S.44 (A16), W2., W4.
- new net A19: P1.54 (A19), U6S.47 (A19)
- new net A20: P1.56 (A20), U6S.48 (A20)
- new net A21: P1.58 (A21), U5L.3 (I3), U6S.50 (A21)
- new net A22: P1.57 (A22), U5L.2 (I2), U6S.51 (A22)
- new net A23: P1.59 (A23), U5L.1 (I1), U6S.52 (A23)
- new net CDAC: P1.15 (CDAC)
- new net EXP: P1.11 (EXP), P1.7 (EXP), P1.9 (EXP)
- new net FC0: P1.31 (FC_{0}), U6S.28 (FC_{0})
- new net FC1: P1.33 (FC_{1}), U6S.27 (FC_{1})
- new net FC2: P1.35 (FC_{2}), U6S.26 (FC_{2})
- new net XRDY: P1.18 (XRDY), RN7-?.7, U5L.8 (I8)
- new net ~{AS}: P1.74 (~{AS}), RN6-.5, U5L.4 (I4), U6S.6 (~{AS})
- new net ~{BERR}: P1.46 (~{BERR}), RN7-.3, RN7-.4, RN7-.5, U6S.22 (~{BERR})
- new net ~{BGACK}: P1.62 (~{BGACK}), RN7-.9, U6S.12 (~{BGACK})
- new net ~{BG}: P1.64 (~{BG}), U6S.11 (~{BG})
- new net ~{BR}: P1.60 (~{BR}), RN7-.8, U6S.13 (~{BR})
- new net ~{C1}: P1.16 (~{C1}), U5L.11 (I10)
- new net ~{C3}: P1.14 (~{C3}), U5L.9 (I9)
- new net ~{DTACK: RN7-.10, U6S.10 (~{DTACK})
- new net ~{DTACK}: P1.66 (~{DTACK})
- new net ~{HLT}: P1.55 (~{HLT}), RN6-.8, U6S.17 (~{HALT}), U7P-.11
- new net ~{LDS}: P1.70 (~{LDS}), RN6-.3, U6S.8 (~{LDS})
- new net ~{OBR}: U5L.5 (I5)
- new net ~{OVR}: P1.17 (~{OVR}), RN7-?.6, U5L.7 (I7)
- new net ~{PALOPE}: P1.20 (~{PALOPE})
- new net ~{PRW}: P1.68 (~{PRW}), RN-.2, U6M-.4, U6S.9 (R/~{W}), W1.
- new net ~{ROME}: U5L.13 (IO7), U5M.7 (I7)
- new net ~{UDS}: P1.72 (~{UDS}), RN6-.4, U6S.7 (~{UDS})
- new net ~{VMA: RN6-.6, U6S.19 (~{VMA})
- new net ~{VMA}: P1.51 (~{VMA}), U6M-.10, U6M-.2
- new net ~{VPA}: P1.48 (~{VPA}), RN7-?.2, U6S.21 (~{VPA})
Other:
- note added: "EVEN"
- note added: "ODD"
- note added: "RN6"
- note added: "RN7"
- note added: "RN8"
- note added: "U2N"
- note added: "U2P"
- moved on the sheet: C1, C10, C100, C101, C102, C103, C104, C105, C106, C107, C108, C109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

Commit message: You know what I worked on!
I'm ALMOST DONE!!!!! (with the Amiga 1000)
Parts:
- added C36, C40, C59, C60, C61, C67, C69, C71, C73, C75, C76, C77: .1, symbol Device:C_Small
- added C62: 10 10V, symbol Device:C_Polarized_Small
- added C68, C70, C72, C74: .001, symbol Device:C_Small
- added C78, C79, C80: 100 16V, symbol Device:C_Polarized_Small
- added FB1, FB2, FB22, FB23, FB24, FB25, FB26, FB27, FB3, FB4, FB41: FERRITE_BEAD, symbol _RS_Commodore_Amiga_1000:FERRITE_BEAD
- added J14: DC POWER, symbol _RS_Commodore_Amiga_1000:CONN_DC_PWR
- added N?: ROM_BRD_NOTE, symbol _RS_Commodore_Amiga_1000:ROM_BRD_NOTE
- added OSC1: 28.63636MHz, symbol Device:Crystal_GND24
- added P1: RAM EXPANSION, symbol _RS_Commodore_Amiga_1000:CONN_RAM
- added R107, R28, R29, R34, R35, R36: 33, symbol Device:R_US
- added R27: 10K, symbol Device:R_US
- added RN2-, RN2-?: 1K, symbol _RS_Commodore_Amiga_1000:RESISTOR_NET_10
- added U1H, U1I: 74F138, symbol _RS_Commodore_Amiga_1000:74F138
- added U2I, U2J: 74F257_U2I_J, Package_DIP:DIP-16_W7.62mm_LongPads, symbol _RS_Commodore_Amiga_1000:74F257_U2I_J
- added U3G: 74LS244_U3G, symbol _RS_Commodore_Amiga_1000:74LS244_U3G
- added U3H: 74LS373_U3H, symbol _RS_Commodore_Amiga_1000:74LS373_U3H
- added U3I: 74LS244_U3I, symbol _RS_Commodore_Amiga_1000:74LS244_U3I
- added U3J: 74LS373_U3J, symbol _RS_Commodore_Amiga_1000:74LS373_U3J
- added U8G-, U8H-, U8I-: 74F74, symbol _RS_Commodore_Amiga_1000:74F74
- added U9G-, U9I-: 74S51, symbol _RS_Commodore_Amiga_1000:74S51
- gave numbers to parts that had none: 1
Connections:
- net +12V: now also C76.1, C79.1, FB2.
- net +5V: now also C36.2, C40.2, C59.2, C60.2, C61.2, C62.2, C75.1, C78.1, FB1., FB22., OSC1.4, R27.1, RN2-., RN2-., RN2-?.2, U9G-.14, U9I-.14
- net -5V: now also C77.1, C80.2, FB3.
- net A19: now also U5M.3 (I3)
- net A20: now also U5M.2 (I2)
- net C1: now also FB26., U1H.4 (E1), U1I.4 (E1)
- net C4: now also FB23., U2I.1 (B/A), U2J.1 (B/A), U3H.11 (L), U3J.11 (L)
- net CCK: now also R35.2
- net CCKQ: now also R34.2
- net CDAC: now also R107.2
- net DAC: now also FB41., R107.1
- net DMAL: now also U5L.15 (IO5), U5M.9 (I9)
- net GND: now also C36.1, C40.1, C59.1, C60.1, C61.1, C62.1, C67.2, C68.2, C69.2, C70.2, C71.2, C72.2, C73.2, C74.2, C75.2, C76.2, C77.2, C78.2, C79.2, C80.1, J14.3 (GND), J14.4 (GND), OSC1.2, U1H.3 (A2), U1H.5 (E2), U1I.3 (A2), U1I.5 (E2), U9G-.4, U9G-.5
- net MA17: now also U1H.1 (A0), U1I.1 (A0)
- net MA18: now also U1H.2 (A1), U1I.2 (A1)
- net TICK: now also FB4.
- net ~{ARW}: now also U5M.1 (I1)
- net ~{BLS}: now also U5L.18 (IO2)
- net ~{C1U}: now also FB25., U8I-.8 (~{Q}), U9I-.2
- net ~{C1}: now also U5M.13 (IO7), FB25.
- net ~{C3}: now also FB24.
- net ~{C4U}: now also U8H-.12 (D), U8H-.6 (~{Q}), U8I-.12 (D), U9I-.10
- net ~{DAE}: now also U5L.14 (IO6), U5M.11 (I10)
- net ~{LDS}: now also U5M.6 (I6)
- net ~{PALOPE}: now also U5M.19 (IO1)
- net ~{PRW}: now also U5M.4 (I4)
- net ~{RE}: now also U5L.16 (IO4), U5M.8 (I8), U2I.15 (OE), U2J.15 (OE)
- net ~{UDS}: now also U5M.5 (I5)
- net ~{VPA}: now also U5L.12 (IO8)
- net ~{XCLKEN}: now also RN2-?., U9G-.13, U9G-.2, U9G-.3
- net ~{XCLK}: now also R27.2, U9G-.9
- net 7MP: now reaches U6S.15 (CLK)
- net 7MP: now also U4A.35 (C7M), R29.1, R29.2, R36.1, R36.2, U9I-.6
- net at C65.1, R14.2, R2.1: now also R5.1
- net at U5N.20 (~{CE}), U5P.20 (~{CE}), W5.: now also U7F-.13, W4.
- net ~{ROM01}: now reaches U5N.22 (~{OE}), U5P.22 (~{OE})
- net ~{ROM01}: now also U5M.12 (IO8)
- net ~{RRW}: now reaches U5M.14 (IO6)
- net LCEN: now reaches U5M.15 (IO5)
- net LCEN: now also U1I.6 (E3)
- net UCEN: now reaches U5M.16 (IO4)
- net UCEN: now also U1H.6 (E3)
- net ~{CDR}: now reaches U5M.17 (I03)
- net ~{CDR}: now also U3H.1 (~{E}), U3J.1 (~{E})
- net ~{CDW}: now reaches U5M.18 (IO2)
- net ~{CDW}: now also U3G.1 (1~{G}), U3G.19 (2~{G}), U3I.1 (1~{G}), U3I.19 (2~{G})
- net ~{QTACK}: now reaches U5L.17 (I03)
- new net: OSC1.3, U9G-.1
- new net: U9G-.10, U9G-.6
- new net: U8G-.3 (C), U9G-.8
- new net: RN2-.3, U8G-.1 (~{R}), U8G-.12 (D), U8H-.1 (~{R}), U8H-.13 (~{R}), U8I-.1 (~{R}), U8I-.13 (~{R})
- new net: FB26., U8I-.2 (D), U8I-.9 (Q)
- new net: RN2-.4, U8G-.10 (~{S}), U8G-.4 (~{S}), U8H-.10 (~{S}), U8H-.4 (~{S}), U8I-.10 (~{S}), U8I-.4 (~{S})
- new net: U8G-.11 (C), U8G-.5 (Q), U8H-.11 (C), U8H-.3 (C), U8I-.11 (C)
- new net: U5N.26 (A14), U5P.26 (A14), W3.
- new net: U5N.20 (~{CE}), U5P.20 (~{CE}), W5.
- new net: FB41., U9I-.8
- new net: U5N.27 (A15), U5P.27 (A15), W1., W2.
- new net: U8H-.2 (D), U8H-.9 (Q)
- new net: U8G-.2 (D), U8G-.6 (~{Q})
- new net +12U: C71.1, C72.1, FB2., J14.2 (+12V)
- new net +5U: C69.1, C70.1, FB1., J14.5 (+5V), J14.6 (+5V)
- new net -5U: C73.1, C74.1, FB3., J14.1 (-5V)
- new net C1U: R35.1, U9I-.4
- new net C2U: U9I-.9
- new net C3U: R34.1, U8I-.5 (Q), U9I-.3
- new net C4U: FB23., U8H-.5 (Q), U9I-.1
- new net MCLK: R28.2
- new net TICKU: C67.1, C68.1, FB4., J14.7 (TICK_{U})
- new net ~{C2U}: R28.1, U8H-.8 (~{Q}), U9I-.13
- new net ~{C3U}: FB24., U8G-.13 (~{R}), U8I-.6 (~{Q}), U9I-.5
- new net ~{RAS}: FB27., P1.23 (~{RAS}), U8G-.9 (Q)
- no-connect marks 11 -> 14
Other:
- note added: "POWER FERRITES (4)"
- note added: "RN2"

Commit message: Amiga 1000 schematic.  COMPLETE!!
Oh thank the MAKER!
Parts:
- added C142: 10 10V TANT, symbol Device:C_Polarized_Small
- added C143..C150: .22 x8, symbol Device:C_Small
- added N2: NOTE_GROUNDS, symbol _RS_Commodore_Amiga_1000:NOTE_GROUNDS
- added R128, R129, R130, R131, R132, R133: 39, symbol Device:R_US
- added RN3: 39, symbol _RS_Commodore_Amiga_1000:RN3
- added unit 9 of RN4
- added RN? (x8): 470, symbol _RS_Commodore_Amiga_1000:RESISTOR_NET_10
- added ROM1: Amiga_1000_RAM_Bank_1, Package_DIP:DIP-18_W7.62mm_LongPads, symbol _RS_Commodore_Amiga_1000:Amiga_1000_RAM_Bank_1
- added ROM2: Amiga_1000_RAM_Bank_2, Package_DIP:DIP-18_W7.62mm_LongPads, symbol _RS_Commodore_Amiga_1000:Amiga_1000_RAM_Bank_2
- RN4: value 100K -> 470
- gave numbers to parts that had none: 3
- renumbered RN- to RN6
Connections:
- net +5V: now also P1.11 (+5V), P1.15 (+5V), P1.29 (+5V), P1.3 (+5V), P1.30 (+5V), P1.7 (+5V), P1.C (+5V), P1.H (+5V), P1.HH (+5V), P1.JJ (+5V), P1.M (+5V), P1.S (+5V), C142.1, C143..C150.2, RN4., RN?., RN?., RN?., RN?., RN?., RN?., RN?., RN?., ROM1.9 (VCC)
- net A1: now also U2I.5 (I0b)
- net A10: now also U2J.6 (I1b)
- net A11: now also U2I.3 (I1a)
- net A12: now also U2J.3 (I1a)
- net A13: now also U2J.13 (I1c)
- net A14: now also U2I.13 (I1c)
- net A15: now also U2J.10 (I1d)
- net A16: now also U2I.10 (I1d)
- net A2: now also U2J.5 (I0b)
- net A3: now also U2I.2 (I0a)
- net A4: now also U2J.2 (I0a)
- net A5: now also U2J.14 (I0c)
- net A6: now also U2I.14 (I0c)
- net A7: now also U2J.11 (I0d)
- net A8: now also U2I.11 (I0d)
- net A9: now also U2I.6 (I1b)
- net D0: now also P1.16 (D0), U3I.3 (2Y4), U3J.8 (4D), ROM1.17 (I/O_{4})
- net D1: now also P1.T (D1), U3I.18 (1Y1), U3J.13 (5D), ROM1.15 (I/O_{3})
- net D10: now also P1.F (D10), U3G.14 (1Y3), U3H.17 (7D), ROM2.2 (I/O_{2})
- net D11: now also P1.6 (D11), U3G.5 (2Y3), U3H.4 (2D), ROM2.3 (I/O_{1})
- net D12: now also P1.4 (D12), U3G.7 (2Y2), U3H.7 (3D), ROM2.17 (I/O_{4})
- net D13: now also P1.D (D13), U3G.16 (1Y2), U3H.14 (6D), ROM2.15 (I/O_{3})
- net D14: now also P1.B (D14), U3G.18 (1Y1), U3H.13 (5D), ROM2.2 (I/O_{2})
- net D15: now also P1.2 (D15), U3G.9 (2Y1), U3H.8 (4D), ROM2.3 (I/O_{1})
- net D2: now also P1.R (D2), U3I.16 (1Y2), U3J.14 (6D), ROM1.2 (I/O_{2})
- net D3: now also P1.14 (D3), U3I.5 (2Y3), U3J.7 (3D), ROM1.3 (I/O_{1})
- net D4: now also P1.12 (D4), U3I.7 (2Y2), U3J.4 (2D), ROM1.17 (I/O_{4})
- net D5: now also P1.N (D5), U3I.14 (1Y3), U3J.17 (7D), ROM1.15 (I/O_{3})
- net D6: now also P1.L (D6), U3I.12 (1Y4), U3J.18 (8D), ROM1.2 (I/O_{2})
- net D7: now also P1.10 (D7), U3I.9 (2Y1), U3J.3 (1D), ROM1.3 (I/O_{1})
- net D8: now also P1.8 (D8), U3G.3 (2Y4), U3H.3 (1D), ROM2.17 (I/O_{4})
- net D9: now also P1.J (D9), U3G.12 (1Y4), U3H.18 (8D), ROM2.15 (I/O_{3})
- net GND: now also P1.1 (DGND), P1.13 (DGND), P1.17 (DGND), P1.22 (DGND), P1.24 (DGND), P1.25 (DGND), P1.27 (DGND), P1.5 (DGND), P1.9 (DGND), P1.A (DGND), P1.BB (DGND), P1.CC (DGND), P1.E (DGND), P1.EE (DGND), P1.K (DGND), P1.P (DGND), P1.U (DGND), P1.Z (DGND), C142.2, ROM1.1 (~{OE}), ROM1.18 (GND), ROM2.1 (~{OE}), ROM2.18 (GND)
- net PD0: now also U3I.11 (2A1), U3J.9 (4Q)
- net PD1: now also U3I.8 (1A4), U3J.12 (5Q)
- net PD10: now also U3G.4 (1A2), U3H.16 (7Q)
- net PD11: now also U3G.15 (2A3), U3H.5 (2Q)
- net PD12: now also U3G.13 (2A2), U3H.6 (3Q)
- net PD13: now also U3G.6 (1A3), U3H.15 (6Q)
- net PD14: now also U3G.8 (1A4), U3H.12 (5Q)
- net PD15: now also U3G.11 (2A1), U3H.9 (4Q)
- net PD2: now also U3I.6 (1A3), U3J.15 (6Q)
- net PD3: now also U3I.13 (2A2), U3J.6 (3Q)
- net PD4: now also U3I.15 (2A3), U3J.5 (2Q)
- net PD5: now also U3I.4 (1A2), U3J.16 (7Q)
- net PD6: now also U3I.2 (1A1), U3J.19 (8Q)
- net PD7: now also U3I.17 (2A4), U3J.2 (1Q)
- net PD8: now also U3G.17 (2A4), U3H.2 (1Q)
- net PD9: now also U3G.2 (1A1), U3H.19 (8Q)
- net RA0: now also U2I.7 (Zb), RN3.7 (R7.1), RN?.9
- net RA1: now also U2J.7 (Zb), RN3.5 (R5.1), RN?.7
- net RA2: now also U2I.4 (Za), RN3.3 (R3.1), RN?.5
- net RA3: now also U2J.4 (Za), RN3.1 (R1.1), RN?.3
- net RA4: now also U2J.12 (Zc), RN3.2 (R2.1), RN?.4
- net RA5: now also U2I.12 (Zc), RN3.4 (R4.1), RN?.6
- net RA6: now also U2J.9 (Zd), RN3.6 (R6.1), RN?.8
- net RA7: now also U2I.9 (Zd), RN3.8 (R8.1), RN4.10
- net ~{RAS}: now also R130.1, R130.2, ROM1.5 (~{RAS})
- net ~{RRW}: now also P1.AA (~{RRW}), R131.1, R131.2, ROM1.4 (~{WE})
- net at U5N.20 (~{CE}), U5P.20 (~{CE}), W5.: now also U7F-.13, W4.
- net DRA4: now reaches P1.18 (DRA4)
- net DRA4: now also ROM2.13 (A4)
- net DRA5: now reaches P1.19 (DRA5)
- net DRA5: now also ROM2.12 (A5)
- net DRA6: now reaches P1.20 (DRA6)
- net DRA6: now also ROM2.11 (A6)
- net DRA7: now reaches P1.21 (DRA7)
- net DRA7: now also ROM2.10 (A7)
- net XN5: now reaches P1.26 (XN5)
- net XN5: now also U1H.13 (O2)
- net XN7: now reaches P1.28 (XN7)
- net XN7: now also U1I.13 (O2)
- net XN4: now reaches P1.DD (XN4)
- net XN4: now also U1H.12 (O3)
- net XN6: now reaches P1.FF (XN6)
- net XN6: now also U1I.12 (O3)
- net DRA3: now reaches P1.V (DRA3)
- net DRA3: now also ROM2.14 (A3)
- net DRA2: now reaches P1.W (DRA2)
- net DRA2: now also ROM2.6 (A2)
- net DRA1: now reaches P1.X (DRA1)
- net DRA1: now also ROM2.7 (A1)
- net DRA0: now reaches P1.Y (DRA0)
- net DRA0: now also ROM2.8 (A0)
- net at U1H.14 (O1): now also R133.1
- net at U1H.15 (O0): now also R129.1
- net at U1I.14 (O1): now also R132.1
- net at U1I.15 (O0): now also R128.1
- new net: R132.2, ROM1.16 (~{CAS})
- new net: U5N.26 (A14), U5P.26 (A14), W3.
- new net: U5N.20 (~{CE}), U5P.20 (~{CE}), W5.
- new net: U5N.27 (A15), U5P.27 (A15), W1., W2.
- new net: RN3.10 (R7.2), ROM1.8 (A0)
- new net: RN3.11 (R6.2), ROM1.11 (A6)
- new net: RN3.12 (R5.2), ROM1.7 (A1)
- new net: RN3.13 (R4.2), ROM1.12 (A5)
- new net: RN3.14 (R3.2), ROM1.6 (A2)
- new net: RN3.15 (R2.2), ROM1.13 (A4)
- new net: RN3.16 (R1.2), ROM1.14 (A3)
- new net: RN3.9 (R8.2), ROM1.10 (A7)
- new net: R133.2, ROM2.16 (~{CAS})
- new net: C143..C150.1, ROM2.9 (VCC)
- new net: ROM1.10 (A7), ROM2.10 (A7)
- new net: ROM1.11 (A6), ROM2.11 (A6)
- new net: ROM1.12 (A5), ROM2.12 (A5)
- new net: ROM1.13 (A4), ROM2.13 (A4)
- new net: ROM1.14 (A3), ROM2.14 (A3)
- new net: R128.2, ROM1.16 (~{CAS})
- new net: ROM1.4 (~{WE}), ROM2.4 (~{WE})
- new net: ROM1.5 (~{RAS}), ROM2.5 (~{RAS})
- new net: ROM1.6 (A2), ROM2.6 (A2)
- new net: ROM1.7 (A1), ROM2.7 (A1)
- new net: ROM1.8 (A0), ROM2.8 (A0)
- new net: ROM1.9 (VCC), ROM2.9 (VCC)
- new net: R129.2, ROM2.16 (~{CAS})
- no-connect marks 14 -> 25
Other:
- note added: "1"
- note added: "RN4 470"
- note removed: "= Shield = Digital = Video = Audio"
- note removed: "SGND = DGND = VGND = AGND ="
- moved on the sheet: C1, C10, C100, C101, C102, C103, C104, C105, C106, C107, C108, C109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
