File: Tandy/TRS-80/Tandy TRS-80 Color Computer 1/Tandy TRS-80 Color Computer 1.kicad_sch (KiCad schematic)
At the start: 43 parts, among them P1 CARTRIDGE CONNECTOR, U1 MC6809E, U10 MC6883, U11 74LS138, U28 MCM68A364, U29 74LS02, U3 MCM68A364, X1 14.31818MHz

Commit message: Started working on schematic sheet 2
Parts:
- added C52: 20pF, symbol Device:C
- added C54 (x2), C56, C78, C79: 0.022µF, symbol Device:C
- added C57, C58: 0.01µF, symbol Device:C
- added CR5, CR6: 1N4148, Diode_THT:D_DO-35_SOD27_P7.62mm_Horizontal, symbol Diode:1N4148
- added L2, L3: 3.3µh, symbol Device:L
- added P2: DIN-4, symbol __Retro_Schematics_Library:DIN-4
- added P3, P4: DIN-6, symbol __Retro_Schematics_Library:DIN-6
- added R10, R22, R28, R29, R48, R51, R52: 10K, symbol Device:R_US
- added R11: 20K, symbol Device:R_US
- added R12: 40.2K, symbol Device:R_US
- added R13: 80.6K, symbol Device:R_US
- added R14: 162K, symbol Device:R_US
- added R15: 324K, symbol Device:R_US
- added R23: 3.9K, symbol Device:R_US
- added R24: 1.5K, symbol Device:R_US
- added R25, R26, R30, R57: 1K, symbol Device:R_US
- added R27, R50: 100Ω 1/2W, symbol Device:R_US
- added R45: 180Ω, symbol Device:R_US
- added R49, R55, R56: 10M, symbol Device:R_US
- added R53, R54: 15K, symbol Device:R_US
- added R72: 100K, symbol Device:R_US
- added S3: CH SELECT, symbol Switch:SW_SPST
- added U14: LM339, symbol __Retro_Schematics_Library:LM339
- added U15: 741C, symbol __Retro_Schematics_Library:741C
- added U2: MC14050B, Package_DIP:DIP-16_W7.62mm_LongPads, symbol __Retro_Schematics_Library:MC14050B
- added unit 1 of U29
- added unit 2 of U29
- added unit 4 of U29
- added U4: MC6821, Package_DIP:DIP-40_W15.24mm_Socket_LongPads, symbol __Retro_Schematics_Library:MC6821
- added U5: UM1285-8 RF Modulator, symbol __Retro_Schematics_Library:UM1285-8 RF Modulator
- added U9: MC14529B, Package_DIP:DIP-16_W7.62mm_LongPads, symbol __Retro_Schematics_Library:MC14529B
- gave numbers to parts that had none: 4
Connections:
- net +12V: now also R45.2, U14.3 (V+), U15.7 (V+)
- net +5V: now also R23.2, R25.1, R26.1, R30.1, R50.2, R53.2, R54.2, R57.2, R72.1, U2.1 (VDD), U4.20 (VCC)
- net -12V: now also U15.4 (V-)
- net A0: now also U4.36 (RS0)
- net A1: now also U4.35 (RS1)
- net D0: now also U4.33 (D0)
- net D1: now also U4.32 (D1)
- net D2: now also U4.31 (D2)
- net D3: now also U4.30 (D3)
- net D4: now also U4.29 (D4)
- net D5: now also U4.28 (D5)
- net D6: now also U4.27 (D6)
- net D7: now also U4.26 (D7)
- net E: now also U4.25 (E)
- net Earth: now also C52.1, C54.1, C54.1, C56.1, C57.1, C58.1, C78.1, C79.1, L2.1, P2.3, P3.3, P3.6, P4.3, P4.6, R24.1, R28.1, R29.1, R51.1, R52.1, S3.2 (B), U14.12 (V-), U2.8 (GND), U29.11, U29.12, U29.2, U29.3, U29.5, U29.6, U4.1 (GND), U5. (GND), U9.11 (Y3)
- net R/~{W}: now also U4.21 (R/~{W})
- net SND: now also U9.12 (Y2)
- net ~{FIRQ}: now also U4.37 (~{IRQB}), U4.38 (~{IRQA})
- net ~{PIA1}: now also U4.23 (~{CS2})
- net ~{RESET}: now also U4.34 (~{RESET})
- new net: CR6.1 (K), R29.2, U14.4 (-)
- new net: C52.2, R10.1, R11.1, R12.1, R13.1, R14.1, R15.1, R72.2, U9.14 (Y0)
- new net: R10.2, U2.10 (OUT_{A})
- new net: R48.1, R49.1, U14.9 (+)
- new net: CR6.2 (A), P2.2
- new net: CR5.1 (K), R28.2, U14.6 (-)
- new net: R12.2, U2.12 (OUT_{A})
- new net: R13.2, U2.4 (OUT_{A})
- new net: U2.5 (IN_{A}), U4.6 (PA4)
- new net: R11.2, U2.6 (OUT_{A})
- new net: U2.7 (IN_{A}), U4.8 (PA6)
- new net: C57.2, L3.2, P4.4
- new net: R22.2, U5.3 (AUDIO), U9.10 (Y)
- new net: U4.19 (CB2), U9.15 (ST_{Y})
- new net: C79.2, P3.2, U9.3 (X1)
- new net: R23.1, R24.2, U15.2 (-)
- new net: U2.11 (IN_{A}), U4.7 (PA5)
- new net: CR5.2 (A), P2.1
- new net: R52.2, R54.1, R56.2, U14.5 (+)
- new net: R48.2, U9.9 (Z)
- new net: C54.2, P3.5, P4.5, R50.1
- new net: C56.2, P4.1, U9.4 (X2)
- new net: C54.2, P4.2, U9.5 (X3)
- new net: P2.4, R27.1
- new net: R27.2, U15.6
- new net: C58.2, L2.2, P3.4
- new net: R51.2, R53.1, R55.2, U14.7 (+)
- new net: R25.2, R55.1, U14.1, U4.40 (CA1)
- new net: R14.2, U2.15 (OUT_{A})
- new net: U2.9 (IN_{A}), U4.9 (PA7)
- new net: C78.2, P3.1, U9.2 (X0)
- new net: R45.1, U5.2 (VCC)
- new net: S3.1 (A), U5.4 (CH_SEL)
- new net: R22.1, U4.11 (PB1)
- new net: U2.3 (IN_{A}), U4.4 (PA2)
- new net: U2.14 (IN_{A}), U4.5 (PA3)
- new net: R15.2, U2.2 (OUT_{A})
- new net CASSDIN: U4.2 (PA0)
- new net CASSMOT: U4.39 (CA2)
- new net CASSOUT: U14.8 (-)
- new net CSN: U9.13 (Y1)
- new net H1: R57.1, U4.22 (CS0), U4.24 (CS1), U9.1 (ST_{X})
- new net JOYIN: R30.2, R49.2, U14.14
- new net LSW: L3.1
- new net RS232IN: R26.2, R56.1, U14.2, U4.10 (PB0)
- new net RS232OUT: U15.3 (+), U4.3 (PA1)
- new net SEL1: U9.6 (A)
- new net SEL2: U9.7 (B)
- no-connect marks 8 -> 11
Other:
- note added: "CARTRIDGE"
- note added: "CASSETTE"
- note added: "D/A (SOUND, JOYSTICK)"
- note added: "GROUNDED CASE"
- note added: "LEFT JOYSTICK"
- note added: "RIGHT JOYSTICK"
- note added: "SPARE GATES"

Commit message: More work on Sheet 2
Parts:
- added C12: 100µF, symbol Device:C
- added C24, C25, C41, C43: 0.1µF, symbol Device:C
- added C42: 0.01µF, symbol Device:C
- added C53: 56pF, symbol Device:C
- added C6: 25µF, symbol Device:C
- added CR16: 1N5228, symbol Device:D_Zener
- added CR8: 1N4002, Diode_THT:D_DO-35_SOD27_P7.62mm_Horizontal, symbol Diode:1N4148
- added Q1: MPS3904, Package_TO_SOT_THT:TO-92_Inline, symbol Transistor_BJT:2N3904
- added R16: 3.9K, symbol Device:R_US
- added R17, R46: 470Ω, symbol Device:R_US
- added R18: 750Ω, symbol Device:R_US
- added R19: 12K, symbol Device:R_US
- added R21: 500Ω, symbol Device:R_Potentiometer_Trim
- added R47: 1.5K, symbol Device:R_US
- added R69: 820Ω, symbol Device:R_US
- added R8: 18K, symbol Device:R_US
- added R9, R?: 150Ω, symbol Device:R_US
- added U12: MC1372, Package_DIP:DIP-14_W7.62mm_LongPads, symbol __Retro_Schematics_Library:MC1372
- added U7: MC6847, Package_DIP:DIP-40_W15.24mm_LongPads, symbol __Retro_Schematics_Library:MC6847
Connections:
- net +12V: now also C24.2, CR16.1 (K)
- net +5V: now also C43.1, C6.1, R9.1, R?.2, U12.11 (VCC), U7.17 (VCC)
- net Earth: now also C12.2, C24.1, C25.2, C41.2, C43.2, C53.1, C6.2, R21.1, R47.2, R69.1, U12.4 (GND), U7.1 (GND)
- net VDG CLK: now also R17.1
- net at U5.1 (VIDEO): now also Q1.1 (E), R46.1, R47.1
- new net: R16.1, R19.2, U12.12 (RF_MOD)
- new net: C12.1, C25.1, CR16.2 (A), Q1.3 (C), R16.2, R69.2
- new net: U12.5 (COLOR_{B}), U7.10 (ɸB)
- new net: U12.7 (COLOR_{A}), U7.11 (ɸA)
- new net: R21.2, R9.2
- new net: R21.3, R46.2, R8.2
- new net: C42.1, R18.1
- new net: R18.2, U12.10 (C)
- new net: CR8.2 (A), R?.1, U12.13 (RFTANK_{1})
- new net: CR8.1 (K), U12.14 (RFTANK_{2})
- new net: C42.2, U12.8 (C_{MOD})
- new net: Q1.2 (B), R19.1, R8.1
- new net 3.58MHz: C53.2, R17.2, U12.2 (OSC), U7.33 (CLK)
- new net BIAS: C41.1, U12.6 (COLOR_{REF}), U7.9 (CHB)
- new net BLACK & WHITE: U12.9 (Y), U7.28 (Y)
- no-connect marks 11 -> 13
Other:
- note added: "COLOR BURST - PORTCH ADJUST PG. 32"
- moved on the sheet: R45

Commit message: Finished Sheet 2
Parts:
- added R44: 4.7K, symbol Device:R_US
- added R68: 10K, symbol Device:R_US
- added TPx, TPx? (x2): TestPoint, symbol Connector:TestPoint
- added U6: 74LS273, symbol __Retro_Schematics_Library:74LS273
Connections:
- net +5V: now also R44.2, R68.2
- net DA0: now also U7.22 (DA0)
- net Earth: now also TPx?.1, U6.10 (GND)
- net H1: now also TPx?.1
- net ~{CART}: now also U4.18 (CB1), R68.1
- net ~{HS}: now also U7.38 (~{HS})
- net ~{RAS}: now also U6.11 (CK)
- net ~{FS}: now reaches U7.12 (~{MS})
- net ~{FS}: now also U7.37 (~{FS})
- net at U7.2 (DD6): now also U7.32 (INV), U6.5 (2Q)
- net at U7.27 (GM2): now also U4.16 (PB6)
- net at U7.29 (GM1): now also U4.15 (PB5)
- net at U7.3 (DD0): now also U6.19 (8Q)
- net at U7.30 (GM0): now also U4.14 (PB4), U7.31 (~{INT}/EXT)
- net at U7.34 (~{A}/S): now also U7.40 (DD7), U6.2 (1Q)
- net at U7.35 (~{A}/G): now also U4.17 (PB7)
- net at U7.39 (CSS): now also U4.13 (PB3)
- net at U7.4 (DD1): now also U6.16 (7Q)
- net at U7.5 (DD2): now also U6.15 (6Q)
- net at U7.6 (DD3): now also U6.12 (5Q)
- net at U7.7 (DD4): now also U6.9 (4Q)
- net at U7.8 (DD5): now also U6.6 (3Q)
- net RAMSZ: now reaches U4.12 (PB2)
- net RAMSZ: now also TPx.1
- new net: R44.1, U6.1 (~{CL})
- new net MD0: U6.18 (8D)
- new net MD1: U6.17 (7D)
- new net MD2: U6.14 (5D)
- new net MD3: U6.13 (3D)
- new net MD4: U6.8 (4D)
- new net MD5: U6.7 (6D)
- new net MD6: U6.4 (2D)
- new net MD7: U6.3 (1D)
Other:
- note added: "16K"
- note added: "4K"
- note added: "COLOR VDG"
- note added: "DATA LATCH"
- note added: "HANDWRITTEN NOTES: (about 7mV/step) 0.25 - 4.7V in 64 steps"
- note added: "HANDWRITTEN NOTES: 1/2 of sound chip (sound selects => joystick selects)"
- note added: "HANDWRITTEN NOTES: 6 Mlte(?) bandwidth/TV Channel Sound - FM Everything else is Arl(?) in TV - black & white Color - phase modulated TV has no sidebands"
- note added: "INPUTS: CA1, CB1 OUTPUTS: CA2, CB2"
- note added: "NOTE FROM OMEGA9380: Again, shown just as it is on the original schematic."
- note added: "PORT A"
- note added: "PORT B"
- note added: "RS232 LEVEL CONVERTERS"
- note added: "SAM SYNC"
- note added: "SHEET 2"
- note added: "VERTICAL SYNC"
- note added: "VIDEO SELECTS"
- moved on the sheet: C12, C24, C25, C41, C42, C43, C52, C53, C54, C56, C57, C58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

Commit message: More work on Sheet 3
Parts:
- added C10: 10,000µF 16V, symbol Device:C_Polarized
- added C11, C13, C83: 0.001µF, symbol Device:C
- added C14: 220µF 16V, symbol Device:C
- added C15: 220µF 16V, symbol Device:C_Polarized
- added C16: 220µF, symbol Device:C_Polarized
- added C17, C18: 1µF, symbol Device:C_Polarized
- added C19: 1µf, symbol Device:C_Polarized_US
- added C20, C21, C22: 0.01µF 1.0 KV, symbol Device:C
- added C27, C? (x4): 1µF, symbol Device:C
- added C30, C76, C77, C80, C81, C? (x6): 0.022µF, symbol Device:C
- added C36 (x2), C37: 0.1µF, symbol Device:C
- added C7: 1800µF 35V, symbol Device:C
- added C82: 0.0022µF, symbol Device:C
- added C9: 470µF 35V, symbol Device:C_Polarized
- added CR10, CR9: 1N982, symbol Device:D_Zener
- added CR11: VM-28, symbol __Retro_Schematics_Library:VM-28
- added CR12, CR13: 3E1, symbol Device:D
- added CR14, CR15: 1N4002, symbol Device:D
- added CR17: 1N4735 6.2V, symbol Device:D_Zener
- added CR4, CR7: 1N4148, symbol Device:D
- added E1, E2, E3, E4, E5, E6, E7, E8: Connector, symbol __Retro_Schematics_Library:Connector
- added F1: 0.7 AMP, symbol Device:Fuse
- added H51: 5060B, symbol __Retro_Schematics_Library:UNKNOWN_H_SYMBOL_COCO
- added H53: 6046, symbol __Retro_Schematics_Library:UNKNOWN_H_SYMBOL_COCO
- added H?: UNKNOWN_H_SYMBOL_COCO, symbol __Retro_Schematics_Library:UNKNOWN_H_SYMBOL_COCO
- added K1: R7336-1, symbol __Retro_Schematics_Library:R7336-1
- added KYBD1: KEYBOARD PBC, symbol __Retro_Schematics_Library:CoCo_1_Keyboard_Matrix
- added P5: DIN-5, symbol __Retro_Schematics_Library:DIN-5
- added Q2: 2N6594, symbol Device:Q_PNP_BEC
- added Q3: TIP29, symbol Device:Q_NPN_BEC
- added Q?: PN2222A, Package_TO_SOT_THT:TO-92_Inline, symbol Transistor_BJT:PN2222A
- added R31, R32, R64: 4.7K, symbol Device:R_US
- added R33, R71: 220Ω, symbol Device:R_US
- added R34: 8.2K, symbol Device:R_US
- added R35: 6.8K, symbol Device:R_US
- added R36, R37: 56K, symbol Device:R_US
- added R38: 15K, symbol Device:R_US
- added R39: 1.5M, symbol Device:R_US
- added R40: 1K, symbol Device:R_US
- added R41: 24K, symbol Device:R_US
- added R42: 75K, symbol Device:R_US
- added R58: 470Ω, symbol Device:R_US
- added R59: 68Ω 1/2W, symbol Device:R_US
- added R60: 1K, symbol Device:R_Potentiometer
- added R61, R63, R67: 1.2K, symbol Device:R_US
- added R62: 3.3K, symbol Device:R_US
- added R65: 560Ω, symbol Device:R_US
- added R66: 0.33Ω 2W, symbol Device:R_US
- added S2: POWER SW, symbol __Retro_Schematics_Library:4PTD_SWITCH
- added T1: TRANSFORMER, symbol __Retro_Schematics_Library:TRFM_COCO1
- added TP10, TP11, TP12, TP4, TP9: Test_Point, symbol __Retro_Schematics_Library:Test_Point
- added U13: 723C, Package_DIP:DIP-14_W7.62mm, symbol __Retro_Schematics_Library:723C
- added unit 3 of U14
- added U17: 78M12, Package_TO_SOT_THT:TO-220-3_Vertical, symbol __Retro_Schematics_Library:78M12
- added U18: 79M12, Package_TO_SOT_THT:TO-220-3_Vertical, symbol __Retro_Schematics_Library:79M12
- added U19: 79L05, Package_TO_SOT_THT:TO-220-3_Vertical, symbol __Retro_Schematics_Library:79L05
- added U8: MC6821, Package_DIP:DIP-40_W15.24mm_Socket_LongPads, symbol __Retro_Schematics_Library:MC6821
Connections:
- net +12V: now also C14.2, C36.2, C77.2, CR14.2 (A), R58.1, TP9., U13.11 (VC), U17. (VO)
- net +5V: now also C16.1, C27.1, C30.1, C83.1, C?.1, C?.1, C?.1, C?.1, C?.1, C?.1, C?.1, C?.1, C?.1, CR17.1 (K), CR7.1 (K), K1., R31.1, R36.2, R37.2, R40.2, R63.1, R66.2, TP12., U13.3 (CS), U8.20 (VCC)
- net -12V: now also C13.2, C15.2, C37.2, C76.1, CR15.1 (K), TP10., U18. (VO)
- net A0: now also U8.36 (RS0)
- net A1: now also U8.35 (RS1)
- net CASSDIN: now also R39.2, R40.1, U14.13
- net CASSMOT: now also R71.2
- net CASSOUT: now also R42.2
- net CSN: now also C?.1, R31.2, R32.1, R33.1, R34.2
- net D0: now also U8.33 (D0)
- net D1: now also U8.32 (D1)
- net D2: now also U8.31 (D2)
- net D3: now also U8.30 (D3)
- net D4: now also U8.29 (D4)
- net D5: now also U8.28 (D5)
- net D6: now also U8.27 (D6)
- net D7: now also U8.26 (D7)
- net E: now also U8.25 (E)
- net Earth: now also C10.2, C13.1, C14.1, C15.1, C16.2, C17.1, C18.1, C19.2, C27.2, C30.2, C36.1, C36.1, C37.1, C7.1, C76.2, C77.1, C81.1, C82.1, C83.2, C9.1, C?.2, C?.2, C?.2, C?.2, C?.2, C?.2, C?.2, C?.2, C?.2, CR17.2 (A), CR4.2 (A), E4., E8., KYBD1.3, P5.2, Q?.1 (E), R32.2, R33.2, R38.1, R41.1, R62.2, R64.2, TP4., U13.7 (V-), U17. (VO), U18. (VO), U19. (VO), U8.1 (GND); no longer L2.1
- net JOYIN: now also U8.9 (PA7)
- net LSW: now also KYBD1.2, U8.3 (PA1)
- net R/~{W}: now also U8.21 (R/~{W})
- net SEL1: now also U8.39 (CA2)
- net SEL2: now also U8.19 (CB2)
- net ~{FS}: now also U8.18 (CB1)
- net ~{HS}: now also U8.40 (CA1)
- net ~{IRQ}: now also U8.37 (~{IRQB}), U8.38 (~{IRQA})
- net ~{RESET}: now also U8.34 (~{RESET})
- net SNDEN: now reaches U4.19 (CB2), U9.15 (ST_{Y})
- new net: C81.2, C?.2, P5.4
- new net: C18.2, R67.1, U19. (VO)
- new net: C82.2, P5.5, R41.2, R42.1
- new net: C11.1, U13.13 (FC)
- new net: C11.2, R63.2, U13.4 (-)
- new net: C17.2, C9.2, CR11. (-), CR15.2 (A), R67.2, U18. (VO)
- new net: C10.1, Q2.2 (E), R59.2, S2.
- new net: Q?.2 (B), R71.1
- new net: K1., Q?.3 (C)
- new net: R37.1, R38.2, R39.1, U14.11 (+)
- new net: C7.2, CR11. (-), CR14.1 (K), U17. (VO)
- new net: E2., S2.
- new net: E2., T1.
- new net: CR10.1 (K), CR9.1 (K)
- new net: C80.1, CR9.2 (A), K1., P5.3
- new net: R60.3, R62.1
- new net: R60.1, R61.1
- new net: R60.2, U13.5 (+)
- new net: R35.1, R36.1, U14.10 (-)
- new net: R61.2, U13.6 (VREF)
- new net: CR12.1 (K), CR13.1 (K), E3.
- new net: CR12.2 (A), T1.
- new net: CR4.1 (K), R34.1, R35.2
- new net: CR13.2 (A), T1.
- new net: C80.2, CR10.2 (A), K1., P5.1
- new net: CR7.2 (A), K1.
- new net: C19.1, R58.2, U13.12 (V+)
- new net: E7., F1.1
- new net: E3., S2.
- new net: CR11. (-), S2. (x2)
- new net: E1., S2.
- new net: Q3.1 (B), R65.1, U13.10 (VO)
- new net: R64.1, R65.2, U13.2 (CL)
- new net: C21.2, C22.1, F1.2, T1.
- new net: C20.1, C22.2, E6., T1.
- new net: E1., T1.
- new net: KYBD1.10, U8.11 (PB1)
- new net: KYBD1.11, U8.12 (PB2)
- new net: KYBD1.12, U8.13 (PB3)
- new net: KYBD1.13, U8.14 (PB4)
- new net: KYBD1.14, U8.15 (PB5)
- new net: KYBD1.15, U8.16 (PB6)
- new net: KYBD1.16, U8.17 (PB7)
- new net: KYBD1.4, U8.4 (PA2)
- new net: KYBD1.5, U8.5 (PA3)
- new net: KYBD1.6, U8.6 (PA4)
- new net: KYBD1.7, U8.7 (PA5)
- new net: KYBD1.8, U8.8 (PA6)
- new net: KYBD1.9, U8.10 (PB0)
- new net: Q2.3 (C), Q3.2 (E), R66.1
- new net: Q2.1 (B), Q3.3 (C), R59.1
- new net -5V: C36.2, TP11., U19. (VO)
- new net AC: E5., E6., E7.
- new net GNDPWR: C20.2, C21.1, E4., E5., E8., T1.
- new net HI: U8.22 (CS0), U8.24 (CS1)
- new net PIA0: U8.23 (~{CS2})
- new net RSW: KYBD1.1, L2.1, U8.2 (PA0)
- no-connect marks 13 -> 14
Other:
- note added: "+12V"
- note added: "+12V REGULATOR"
- note added: "+5V REG"
- note added: "-12V REGULATOR"
- note added: "-5V REGULATOR"
- note added: "1.35 AMPS"
- note added: "100MA"
- note added: "100µA"
- note added: "16K RAM BIAS"
- note added: "2N6-594"
- note added: "400MA"
- note added: "5%, 1% +5 REG NOT EXCHANGEABLE"
- note added: "5072B & 5071B"
- note added: "BRIDGE RECTIFIER ~20V"
- note added: "H52"
- note added: "H54"
- note added: "HANDWRITTEN NOTE: 5V relays are weak"
- note added: "HANDWRITTEN NOTE: signals are logoing (sic)"
- note added: "LIMITING -ABOVE +6.2V"
- note added: "NOTE FROM OMEGA9380 On the original schematic, it looks like L2 connects to nothing. LSW connects to L3 and there is a reference on Sheet 3 to RSW. I am assuming that there was supposed to be a reference to RSW connected to L2."
- note added: "ON OLD SETS USED TO ADJUST +5V"
- note added: "PIA"
- note added: "POWER SUPPLY"
- note added: "SINGLE BIT SOUND"
- note added: "TRANSFORMER ASSEMBLY"
- moved on the sheet: C54

Commit message: Finished schematic for CoCo 1
Parts:
- added C23, C29, C31, C32, C33, C35, C39, C45, C46, C47, C48, C49, C61, C62, C63, C64, C65, C66, C67, C68, C69, C70, C71, C72: 1µF, symbol Device:C
- added C8: 100µF, symbol Device:C
- added U16: 74LS244, symbol __Retro_Schematics_Library:74LS244
- added U20, U21, U22, U23, U24, U25, U26, U27: MCM4027A, Package_DIP:DIP-16_W7.62mm_LongPads, symbol __Retro_Schematics_Library:MCM4027A
Connections:
- net A2 is gone; now on net MA2: P1.21 (Pin_21), U1.10 (A2), U10.18 (A2), U3.6 (A2)
- net A3 is gone; now on net MA3: P1.22 (Pin_22), U1.11 (A3), U10.19 (A3), U3.5 (A3)
- net A4 is gone; now on net MA4: P1.23 (Pin_23), U1.12 (A4), U10.21 (A4), U3.4 (A4)
- net A5 is gone; now on net MA5: P1.24 (Pin_24), U1.13 (A5), U10.22 (A5), U3.3 (A5)
- net A6 is gone; now on net MA6: P1.25 (Pin_25), U1.14 (A6), U10.23 (A6), U3.2 (A3)
- net MA0 is gone; now on net A0: R75.10
- net MA1 is gone; now on net A1: R76.1
- net +12V: now also C32.2, C39.2, C46.2, C49.2, C62.2, C65.2, C68.2, C71.2, C8.2, U20.8 (VDD), U21.8 (VDD), U22.8 (VDD), U23.8 (VDD), U24.8 (VDD), U25.8 (VDD), U26.8 (VDD), U27.8 (VDD)
- net +5V: now also C31.2, C35.2, C45.2, C48.2, C61.2, C64.2, C67.2, C70.2, U16.20 (VCC), U20.9 (VCC), U21.9 (VCC), U22.9 (VCC), U23.9 (VCC), U24.9 (VCC), U25.9 (VCC), U26.9 (VCC), U27.9 (VCC)
- net -5V: now also C23.2, C29.2, C33.2, C47.2, C63.2, C66.2, C69.2, C72.2, U20.1 (VBB), U21.1 (VBB), U22.1 (VBB), U23.1 (VBB), U24.1 (VBB), U25.1 (VBB), U26.1 (VBB), U27.1 (VBB)
- net A0: now also U20.5 (A0), U21.5 (A0), U22.5 (A0), U23.5 (A0), U24.5 (A0), U25.5 (A0), U26.5 (A0), U27.5 (A0)
- net A1: now also U20.7 (A1), U21.7 (A1), U22.7 (A1), U23.7 (A1), U24.7 (A1), U25.7 (A1), U26.7 (A1), U27.7 (A1)
- net D0: now also U16.3 (1Y), U20.2 (D)
- net D1: now also U16.18 (2Y), U21.2 (D)
- net D2: now also U16.5 (3Y), U22.2 (D)
- net D3: now also U16.16 (4Y), U23.2 (D)
- net D4: now also U16.7 (5Y), U24.2 (D)
- net D5: now also U16.14 (6Y), U25.2 (D)
- net D6: now also U16.9 (7Y), U26.2 (D)
- net D7: now also U16.12 (8Y), U27.2 (D)
- net Earth: now also C23.1, C29.1, C31.1, C32.1, C33.1, C35.1, C39.1, C45.1, C46.1, C47.1, C48.1, C49.1, C61.1, C62.1, C63.1, C64.1, C65.1, C66.1, C67.1, C68.1, C69.1, C70.1, C71.1, C72.1, C8.1, U16.10 (GND), U20.16 (VSS), U21.16 (VSS), U22.16 (VSS), U23.16 (VSS), U24.16 (VSS), U25.16 (VSS), U26.16 (VSS), U27.16 (VSS)
- net MA2: now also U20.6 (A2), U21.6 (A2), U22.6 (A2), U23.6 (A2), U24.6 (A2), U25.6 (A2), U26.6 (A2), U27.6 (A2)
- net MA3: now also U20.12 (A3), U21.12 (A3), U22.12 (A3), U23.12 (A3), U24.12 (A3), U25.12 (A3), U26.12 (A3), U27.12 (A3)
- net MA4: now also U20.11 (A4), U21.11 (A4), U22.11 (A4), U23.11 (A4), U24.11 (A4), U25.11 (A4), U26.11 (A4), U27.11 (A4)
- net MA5: now also U20.10 (A5), U21.10 (A5), U22.10 (A5), U23.10 (A5), U24.10 (A5), U25.10 (A5), U26.10 (A5), U27.10 (A5)
- net MA6: now also U20.13 (A6), U21.13 (A6), U22.13 (A6), U23.13 (A6), U24.13 (A6), U25.13 (A6), U26.13 (A6), U27.13 (A6)
- net MD0: now also U16.17 (1A), U20.14 (Q)
- net MD1: now also U16.2 (2A), U21.14 (Q)
- net MD2: now also U16.15 (3A), U22.14 (Q)
- net MD3: now also U16.4 (4A), U23.14 (Q)
- net MD4: now also U16.13 (5A), U24.14 (Q)
- net MD5: now also U16.6 (6A), U25.14 (Q)
- net MD6: now also U16.11 (7A), U26.14 (Q)
- net MD7: now also U16.8 (8A), U27.14 (Q)
- net ~{CAS}: now also U20.15 (~{CAS}), U21.15 (~{CAS}), U22.15 (~{CAS}), U23.15 (~{CAS}), U24.15 (~{CAS}), U25.15 (~{CAS}), U26.15 (~{CAS}), U27.15 (~{CAS})
- net ~{MRD}: now also U16.1 (1~{G}), U16.19 (2~{G})
- net ~{RAS}: now also U20.4 (~{RAS}), U21.4 (~{RAS}), U22.4 (~{RAS}), U23.4 (~{RAS}), U24.4 (~{RAS}), U25.4 (~{RAS}), U26.4 (~{RAS}), U27.4 (~{RAS})
- net ~{WE}: now also U20.3 (~{WE}), U21.3 (~{WE}), U22.3 (~{WE}), U23.3 (~{WE}), U24.3 (~{WE}), U25.3 (~{WE}), U26.3 (~{WE}), U27.3 (~{WE})
- net at E2.: now also T1.; no longer S2.
- net at S2.: now also E1.; no longer CR11. (-)
- net at E1.: now also T1.; no longer S2.
- new net: E2., S2.
- new net: CR11. (-), S2.
Other:
- note added: "HANDWRITTEN NOTE: Write to mem is directly off data lines Refresh during horizontal sync"
- note added: "SHEET 3"
- moved on the sheet: C1, C10, C11, C12, C13, C14, C15, C16, C17, C18, C19, C20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
