File: Commodore/Commodore 64/Commodore 64.kicad_sch (KiCad schematic)
At the start: 41 parts, among them CN6 CARTRIDGE/EXPANSION (44PIN FE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, U12,U24,U11,U23,U10,U22,U9,U21 4146_U9..U12,U21..U24, U13 74LS257_U13, U14 74LS258_U14, U16 4066_U16, U19 6567_U19, U25 74LS257_U25, U26 74LS373_U26, U27 74LS08, U3 2364_BASIC_ROM_U3, U4 2364_KERNAL_ROM_U4, U5 2332_CHAR_ROM_U5, U6 2114-30L_U6, U8 7406N

Commit message: Finished Sheet 1 C64 Schematic #251138
Parts:
- added C10, C11: 470pF, symbol Device:C_Small
- added C12, C16, C31, C33, C4, C49, C5, C50, C51, C52, C6: .1, symbol Device:C_Small
- added C13, C15, C17, C34, C62: 10 25V, symbol Device:C_Polarized_Small
- added C203, C205: 220pF, symbol Device:C_Small
- added C204: 150pF, symbol Device:C_Small
- added C37: 1000 pF, symbol Device:C_Small
- added C48, C93: 1800pF, symbol Device:C_Small
- added CN5: AUDIO/VIDEO (8PIN FEMALE DIN), symbol Commodore_64:CONN_AV_CN5
- added FB10, FB11, FB13, FB14, FB15, FB29, FB4: FerriteBead_Small, symbol Device:FerriteBead_Small
- added J99: RF_OUT, symbol Connector:Conn_Coaxial
- added JP99: Jumper_2_Bridged, symbol Jumper:Jumper_2_Bridged
- added Q8: 2SC1815, Package_TO_SOT_THT:TO-92_Inline, symbol Transistor_BJT:2SC1815
- added R38, R6: 1K, symbol Device:R_US
- added R42: 82Ω, symbol Device:R_US
- added R51: 1.5K, symbol Device:R_US
- added R7: 10K, symbol Device:R_US
- added RF1: RF_MODULATOR, symbol Commodore_64:RF_MODULATOR
- added RP4: 3.3K, symbol Commodore_64:RESISTOR_PACK_10PIN_RN4
- added U15: 74LS139_U15, symbol Commodore_64:74LS139_U15
- added U18: 6581_SID_U18, Package_DIP:DIP-28_W15.24mm_LongPads, symbol Commodore_64:6581_SID_U18
- added unit 4 of U27
- added unit 3 of U27
- gave numbers to parts that had none: 3
Connections:
- net +12V: now also C52.2, C62.1, FB11.2, Q8.2 (C)
- net +5V: now also CN6.2 (+5V), CN6.3 (+5V), U17.28 (VCC), U3.24 (VCC), U4.24 (VCC), U5.21 (CS_{2}), U5.24 (VCC), C17.2, C31.1, C33.1, C34.1, C4.2, C49.2, C5.2, C6.2, FB10.2, R51.1, RP4.1, RP4.1, RP4.1, RP4.1, U15.16 (VCC)
- net A0: now also U3.8 (A0), U4.8 (A0), U5.8 (A0), U18.9 (A0)
- net A1: now also U3.7 (A1), U4.7 (A1), U5.7 (A1), U18.10 (A1)
- net A10: now also U3.19 (A10), U4.19 (A10), U5.19 (A10), U15.2 (A0)
- net A11: now also U3.18 (A11), U4.18 (A11), U5.18 (A11), U15.3 (A1)
- net A12: now also U17.27 (I8), U3.21 (A12), U4.21 (A12)
- net A13: now also U17.2 (I7)
- net A14: now also U17.3 (I6)
- net A15: now also U17.4 (I5)
- net A2: now also U3.6 (A2), U4.6 (A2), U5.6 (A2), U18.11 (A2)
- net A3: now also U3.5 (A3), U4.5 (A3), U5.5 (A3), U18.12 (A3)
- net A4: now also U3.4 (A4), U4.4 (A4), U5.4 (A4), U18.13 (A4)
- net A5: now also U3.3 (A5), U4.3 (A5), U5.3 (A5)
- net A6: now also U3.2 (A6), U4.2 (A6), U5.2 (A6)
- net A7: now also U3.1 (A7), U4.1 (A7), U5.1 (A7)
- net A8: now also U3.23 (A8), U4.23 (A8), U5.23 (A8), U15.14 (A0)
- net A9: now also U3.22 (A9), U4.22 (A9), U5.22 (A9), U15.13 (A1)
- net D0: now also CN6.21 (D0), U3.9 (D0), U4.9 (D0), U5.9 (D0), U18.15 (D0)
- net D1: now also CN6.20 (D1), U3.10 (D1), U4.10 (D1), U5.10 (D1), U18.16 (D1)
- net D2: now also CN6.19 (D2), U3.11 (GND), U4.11 (GND), U5.11 (GND), U18.17 (D2)
- net D3: now also CN6.18 (D3), U3.13 (D3), U4.13 (D3), U5.13 (D3), U18.18 (D3)
- net D4: now also CN6.17 (D4), U3.14 (D4), U4.14 (D4), U5.14 (D4), U18.19 (D4)
- net D5: now also CN6.16 (D5), U3.15 (D5), U4.15 (D5), U5.15 (D5), U18.20 (D5)
- net D6: now also CN6.15 (D6), U3.16 (D6), U4.16 (D6), U5.16 (D6), U18.21 (D6)
- net D7: now also CN6.14 (D7), U3.17 (D7), U4.17 (D7), U5.17 (D7), U18.22 (D7)
- net GND: now also CN6.1 (GND), CN6.22 (GND), CN6.A (GND), CN6.Z (GND), U17.14 (GND), U17.19 (~{OE}), U3.11 (GND), U4.11 (GND), U5.11 (GND), U6.9 (GND), C15.2, C16.1, C17.1, C203.1, C204.1, C205.1, C31.2, C33.2, C34.2, C37.1, C4.1, C48.1, C49.1, C5.1, C50.1, C51.1, C52.1, C6.1, C62.2, C93.2, CN5.2 (GND), J99.2 (Ext), JP99.2 (B), R38.2, R6.2, RF1.10 (CASE_GND), U15.8 (GND), U18.14 (GND)
- net ~{AEC}: now also U17.25 (I10), U27.12
- net ~{IRQ}: now also RP4.3
- net ~{VA14}: now also U17.5 (I4)
- net ɸ0: now also FB29.2; no longer U19.17 (ɸ0_{OUT})
- net VA13: now reaches U12,U24,U11,U23,U10,U22,U9,U21.10 (MA5), U19.29 (A5/A13), U26.18 (D5)
- net VA13: now also U17.21 (I14)
- net VA12: now reaches U12,U24,U11,U23,U10,U22,U9,U21.11 (MA4), U19.28 (A4/A12), U26.17 (D4)
- net VA12: now also U17.20 (I15)
- net ~{CASRAM}: now reaches U12,U24,U11,U23,U10,U22,U9,U21.15 (~{CAS})
- net ~{CASRAM}: now also U17.18 (F0), C204.2, R42.1, R42.2
- net at U12,U24,U11,U23,U10,U22,U9,U21.3 (~{WE}), U19.11 (R/~{W}): now also U18.7 (R/~{W})
- net ~{DMA: now reaches U27.4
- net ~{DMA: now also CN6.13 (~{DMA}), RP4.10, U27.10
- net ~{VIC}: now reaches U19.10 (~{CS})
- net ~{VIC}: now also U15.4 (O0)
- net BA: now reaches CN6.12 (BA), U19.12 (BA)
- net BA: now also U17.26 (I9), U27.9
- net at U19.14 (COLOR): now also FB14.1
- net at U19.15 (SYNC/LUM): now also FB15.1
- net ~{CAS}: now reaches U13.1 (~{SELA}), U14.1 (~{SELA}), U19.19 (~{CAS}), U25.1 (~{SELA})
- net ~{CAS}: now also U17.9 (I0), C203.2
- net ~{ROMH}: now reaches U17.10 (F7)
- net ~{ROMH}: now also CN6.11 (~{ROML}), CN6.B (~{ROMH}), U17.11 (F6)
- net ~{I/O}: now reaches U17.12 (F5)
- net ~{I/O}: now also U15.1 (E)
- net GR/~{W}: now reaches U17.13 (F4)
- net GR/~{W}: now also U6.10 (~{WE})
- net ~{CHAROM}: now reaches U17.15 (F3)
- net ~{CHAROM}: now also U5.20 (~{CS_{1}})
- net ~{KERNAL}: now reaches U17.16 (F2)
- net ~{KERNAL}: now also U4.20 (~{CS})
- net ~{BASIC}: now reaches U17.17 (F1)
- net ~{BASIC}: now also U3.20 (~{CS})
- net ~{GAME}: now reaches U17.22 (I13)
- net ~{GAME}: now also CN6.8 (~{GAME}), RP4.7
- net ~{EXROM}: now reaches U17.23 (I12)
- net ~{EXROM}: now also CN6.9 (~{EXROM}), RP4.9
- net R/~{W}: now reaches U17.24 (I11)
- net R/~{W}: now also CN6.5 (R/~{W}), R51.2
- net ~{CHAREN}: now reaches U17.6 (I3)
- net ~{HIRAM}: now reaches U17.7 (I2)
- net ~{LORAM}: now reaches U17.8 (I1)
- net at U6.8 (~{CS}): now also U27.11
- net ~{I/O_{2}}: now reaches CN6.10 (~{I/O_{2}})
- net ~{I/O_{2}}: now also U15.9 (O3)
- net ~{I/O_{1}}: now reaches CN6.7 (~{I/O_{1}})
- net ~{I/O_{1}}: now also U15.10 (O2)
- net ~{RESET}: now reaches CN6.C (~{RESET})
- net ~{RESET}: now also FB4.1, FB4.2, U18.5 (~{RES})
- net ɸ2: now reaches CN6.E (ɸ2)
- net ɸ2: now also U18.6 (ɸ2)
- new net: C13.1, C205.2, Q8.1 (E), R38.1
- new net: C51.2, FB11.1, U18.28 (VDD)
- new net: FB15.2, RF1.2 (SYNC+LUM_{IN})
- new net: C50.2, FB10.1, U18.25 (VCC)
- new net: FB14.2, RF1.3 (COLOR_{IN})
- new net: C13.2, CN5.3 (AUD_OUT), RF1.4 (AUDIO)
- new net: CN5.4 (COMP_VID), RF1.5 (COMP_{OUT})
- new net: CN5.1 (LUM), RF1.6 (SYNC+LUM_{OUT})
- new net: CN5.6 (COLOR), RF1.7 (COLOR_{OUT})
- new net: JP99.1 (A), RF1.8 (ICS)
- new net: J99.1 (In), RF1.9 (RF_OUT)
- new net: C37.2, Q8.3 (B), R7.2
- new net: C10.1, U18.2 (CAP_{1B})
- new net: C10.2, U18.1 (CAP_{1A})
- new net: FB29.1, U19.17 (ɸ0_{OUT})
- new net: FB13.1, R6.1, U18.27 (AUD_{OUT})
- new net: FB13.2, R7.1
- new net: C12.1, U18.26 (EXT_{IN})
- new net: C12.2, CN5.5 (AUD_IN)
- new net: C11.2, U18.3 (CAP_{2A})
- new net: C11.1, U18.4 (CAP_{2B})
- new net +9V: C15.1, C16.2, RF1.1 (+B)
- new net POT_{X}: C48.2, U18.23 (POT_{X})
- new net POT_{Y}: C93.1, U18.24 (POT_{Y})
- new net RDY: U27.8
- new net ~{CIA1}: U15.12 (O0)
- new net ~{CIA2}: U15.11 (O1)
- new net ~{CLAS}: U15.15 (E), U15.7 (O3)
- new net ~{COLOR}: U15.6 (O2), U27.13
- new net ~{NMI}: CN6.D (~{NMI})
- new net ~{SID}: U15.5 (O1), U18.8 (~{CS})
- no-connect marks 0 -> 4
Other:
- note added: "(8000-9FFF)"
- note added: "(A000-BFFF OR E000-FFFF)"
- note added: "(DE00-DEFF:Z80 ON)"
- note added: "(DF00-DFFF:DISK)"
- note added: "RP4 3.3K"
- note added: "SEE NOTE 5"
- note added: "SHEET 1"
- note added: "UNREG"
- moved on the sheet: C101, C14, C25, C26, C27, C28, C29, C30, C32, C40, C41, C42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

Commit message: Working on C64 Sheet 2
Parts:
- added C22, C3, C47, C9, C96, C?: .1, symbol Device:C_Small
- added C23: 360pF, symbol Device:C_Small
- added C38: 51pF, symbol Device:C_Small
- added C8: 10 25V, symbol Device:C_Polarized_Small
- added CN1: KEYBOARD, symbol Commodore_64:CONN_KEYBOARD_CN1
- added CN2: USER PORT, symbol Commodore_64:CONN_USER_CN2
- added CN4: SERIAL BUS, symbol Commodore_64:CONN_SERIAL_CN4
- added CN8: CONTROL PORT 2, symbol Commodore_64:CONN_CTRL2_CN8
- added CN9: CONTROL PORT 1, symbol Commodore_64:CONN_CTRL1_CN9
- added CR100, CR101, CR102, CR103: D_Small, symbol Device:D_Small
- added FB18, FB5, FB87, FB88, FB89: FerriteBead_Small, symbol Device:FerriteBead_Small
- added R28, R29, R30: 1K, symbol Device:R_US
- added R33: 47K, symbol Device:R_US
- added R35: 470K, symbol Device:R_US
- added R41: 1M, symbol Device:R_US
- added RP3: 3.3K, symbol Commodore_64:RESISTOR_PACK_8PIN_RN3
- added unit 3 of RP4
- added unit 4 of RP4
- added unit 7 of RP4
- added unit 5 of RP4
- added U1: 6526_CIA_U1, Package_DIP:DIP-40_W15.24mm_LongPads, symbol Commodore_64:6526_CIA_U1
- added U2: 6526_CIA_U2, Package_DIP:DIP-40_W15.24mm_LongPads, symbol Commodore_64:6526_CIA_U2
- added U20: LM556_U20, symbol Commodore_64:LM556_U20
- added U28: 4066, Package_DIP:DIP-14_W7.62mm_LongPads, symbol Commodore_64:4066_U28
- added U7: 6510_MPU_U7, Package_DIP:DIP-40_W15.24mm_LongPads, symbol Commodore_64:6510_MPU_U7
- added unit 1 of U8
- added unit 6 of U8
- added unit 3 of U8
- added unit 5 of U8
Connections:
- net +5V: now also C22.1, C3.2, C47.1, C8.1, C9.2, C96.2, C?.2, CN1.4 (+5V), CN2.2 (+5V), CR100.1 (K), CR102.1 (K), FB18.1, R28.1, R29.1, R30.1, R33.1, R35.2, R41.1, RP3.1, RP3.1, RP3.1, RP3.1, RP3.1, RP3.1, RP3.1, RP4.1, RP4.1, RP4.1, RP4.1, U1.20 (VCC), U2.20 (VCC), U20.4 (RST_{1}), U28.14 (VDD), U7.6 (VCC), U8.14
- net A0: now also U1.38 (RS0), U2.38 (RS0), U7.7 (A0)
- net A1: now also U1.37 (RS1), U2.37 (RS1), U7.8 (A1)
- net A10: now also U7.17 (A10)
- net A11: now also U7.18 (A11)
- net A12: now also RP4.8, U7.19 (A12)
- net A13: now also RP4.6, U7.20 (A13)
- net A14: now also RP4.5, U7.22 (A14)
- net A15: now also RP4.4, U7.23 (A15)
- net A2: now also U1.36 (RS2), U2.36 (RS2), U7.9 (A2)
- net A3: now also U1.35 (RS3), U2.35 (RS3), U7.10 (A3)
- net A4: now also U7.11 (A4)
- net A5: now also U7.12 (A5)
- net A6: now also U7.13 (A6)
- net A7: now also U7.14 (A7)
- net A8: now also U7.15 (A8)
- net A9: now also U7.16 (A9)
- net BTN_{A}/LP: now also CN1.8 (ROW_{4}), CN9.6 (BTN_{A}/LP), U1.14 (PB4)
- net D0: now also U1.33 (DB0), U2.33 (DB0), U7.37 (D0)
- net D1: now also U1.32 (DB1), U2.32 (DB1), U7.36 (D1)
- net D2: now also U1.31 (DB2), U2.31 (DB2), U7.35 (D2)
- net D3: now also U1.30 (DB3), U2.30 (DB3), U7.34 (D3)
- net D4: now also U1.29 (DB4), U2.29 (DB4), U7.33 (D4)
- net D5: now also U1.28 (DB5), U2.28 (DB5), U7.32 (D5)
- net D6: now also U1.27 (DB6), U2.27 (DB6), U7.31 (D6)
- net D7: now also U1.26 (DB7), U2.26 (DB7), U7.30 (D7)
- net GND: now also C22.2, C23.2, C3.1, C47.2, C8.2, C9.1, C96.1, C?.1, CN1.1 (GND), CN2.1 (GND), CN2.12 (GND), CN2.A (GND), CN2.N (GND), CN4.2 (GND), CN8.8 (GND), CN9.8 (GND), CR101.2 (A), CR103.2 (A), U1.1 (GND), U2.1 (GND), U28.7 (GND), U7.21 (GND), U8.7
- net POT_{X}: now also U28.2 (Z_{0}), U28.9 (Z_{2})
- net POT_{Y}: now also U28.10 (Z_{3}), U28.3 (Z_{1})
- net RDY: now also U7.2 (RDY)
- net R/~{W}: now also U1.22 (R/~{W}), U2.22 (R/~{W}), U7.38 (R/~{W})
- net ~{CIA1}: now also U1.23 (~{CS})
- net ~{CIA2}: now also U2.23 (~{CS})
- net ~{IRQ}: now also U1.21 (~{IRQ}), U7.3 (~{IRQ})
- net ~{NMI}: now also RP3.3, U2.21 (~{IRQ}), U7.4 (~{NMI}), U8.6
- net ~{RESET}: now also CN2.3 (~{RESET}), CN4.6 (~{RESET}), U1.34 (~{RES}), U2.34 (~{RES}), U7.40 (~{RES})
- net ~{VA14}: now also U2.2 (PA0)
- net ~{VA15}: now also U2.3 (PA1)
- net ɸ2: now also FB5.1, FB5.2, U1.25 (ɸ2), U2.25 (ɸ2), U7.39 (ɸ2)
- new net: C23.1, R33.2, U20.1 (DIS_{1}), U20.2 (THR_{1})
- new net: CN8.7 (+5V), CN9.7 (+5V), FB18.2
- new net: U1.19 (TOD), U2.19 (TOD)
- new net: C38.2, R35.1, U20.6 (TRIG_{1})
- new net: U20.5 (OUT_{1}), U8.5
- new net ATN: CN2.9 (ATN), CN4.3 (ATN), FB87.1, FB87.2, R28.2, U8.12
- new net ATN_OUT: U2.5 (PA3), U8.13
- new net BTN_{B}: CN1.16 (COL_{4}), CN8.6 (BTN_{B}), U1.6 (PA4)
- new net CASS RD: CN4.1 (~{SRQIN}), RP3.4, U1.24 (~{FLAG})
- new net CLK: CN4.4 (CLK), CR102.2 (A), CR103.1 (K), FB89.1, FB89.2, R30.2, U2.8 (PA6), U8.10
- new net CLK_OUT: U2.6 (PA4), U8.11
- new net CNT1: CN2.4 (CNT1), RP3.5, U1.40 (CNT)
- new net CNT2: CN2.6 (CNT2), RP3.7, U2.40 (CNT)
- new net COL_{0}: CN1.13 (COL_{0}), CN8.1 (JOY_{B}0), U1.2 (PA0)
- new net COL_{1}: CN1.19 (COL_{1}), CN8.2 (JOY_{B}1), U1.3 (PA1)
- new net COL_{2}: CN1.18 (COL_{2}), CN8.3 (JOY_{B}2), U1.4 (PA2)
- new net COL_{3}: CN1.17 (COL_{3}), CN8.4 (JOY_{B}3), U1.5 (PA3)
- new net COL_{5}: CN1.15 (COL_{5}), U1.7 (PA5)
- new net COL_{6}: CN1.14 (COL_{6}), U1.8 (PA6), U28.12 (E_{3}), U28.6 (E_{2})
- new net COL_{7}: CN1.20 (COL_{7}), U1.9 (PA7), U28.13 (E_{0}), U28.5 (E_{1})
- new net DATA: CN4.5 (DATA), CR100.2 (A), CR101.1 (K), FB88.1, FB88.2, R29.2, U2.9 (PA7), U8.2
- new net DATA_OUT: U2.7 (PA5), U8.1
- new net JOY_{A}0: CN1.12 (ROW_{0}), CN9.1 (JOY_{A}0), U1.10 (PB0)
- new net JOY_{A}1: CN1.11 (ROW_{1}), CN9.2 (JOY_{A}1), U1.11 (PB1)
- new net JOY_{A}2: CN1.10 (ROW_{2}), CN9.3 (JOY_{A}2), U1.12 (PB2)
- new net JOY_{A}3: CN1.5 (ROW_{3}), CN9.4 (JOY_{A}3), U1.13 (PB3)
- new net PA2: CN2.M (PA2), U2.4 (PA2)
- new net PB0: CN2.C (PB0), U2.10 (PB0)
- new net PB1: CN2.D (PB1), U2.11 (PB1)
- new net PB2: CN2.E (PB2), U2.12 (PB2)
- new net PB3: CN2.F (PB3), U2.13 (PB3)
- new net PB4: CN2.H (PB4), U2.14 (PB4)
- new net PB5: CN2.J (PB5), U2.15 (PB5)
- new net PB6: CN2.K (PB6), U2.16 (PB6)
- new net PB7: CN2.L (PB7), U2.17 (PB7)
- new net POT_{A}X: CN9.9 (POT_{A}X), U28.8 (Y_{2})
- new net POT_{A}Y: CN9.5 (POT_{A}Y), U28.11 (Y_{3})
- new net POT_{B}X: CN8.9 (POT_{B}X), U28.1 (Y_{0})
- new net POT_{B}Y: CN8.5 (POT_{B}Y), U28.4 (Y_{1})
- new net ROW_{5}: CN1.7 (ROW_{5}), U1.15 (PB5)
- new net ROW_{6}: CN1.6 (ROW_{6}), U1.16 (PB6)
- new net ROW_{7}: CN1.9 (ROW_{7}), U1.17 (PB7)
- new net SP1: CN2.5 (SP1), RP3.6, U1.39 (SP)
- new net SP2: CN2.7 (SP2), RP3.8, U2.39 (SP)
- new net ~{FLAG2}: CN2.B (~{FLAG2}), RP3.2, U2.24 (~{FLAG})
- new net ~{PC2}: CN2.8 (~{PC2}), U2.18 (~{PC})
- new net ~{RESTORE}: C38.1, CN1.3 (~{RESTORE}), R41.2
- no-connect marks 4 -> 7
Other:
- note added: "(20-PIN MALE)"
- note added: "(24-PIN MALE EDGE)"
- note added: "(6-PIN FEMALE DIN)"
- note added: "(MALE DB9)"
- note added: "RP3 3.3K"

Commit message: More C64 schematic work
Parts:
- added C105, C18, C39, C56, C68, C74, C82, C84: .1, symbol Device:C_Small
- added C107: NOTE 2, symbol Device:C_Polarized_Small
- added C108, C24: 10 25V, symbol Device:C_Polarized_Small
- added C36: 20pF 50V, symbol Device:C_Small
- added C70: NOTE 2, symbol Device:C_Small
- added C83: 82pF 50V ±5%, symbol Device:C_Small
- added C85: .47, symbol Device:C_Small
- added C86: NOTE 8, symbol Device:C_Small
- added CN3: CASSETTE, symbol Commodore_64:CONN_CASSETTE_CN3
- added CR2: 1.5V IN755, symbol Device:D_Zener
- added E1: JUMPER_SELECT, symbol Commodore_64:JUMPER_SELECT
- added FB1, FB16, FB17, FB2: FerriteBead_Small, symbol Device:FerriteBead_Small
- added Q1, Q2, Q7: 2SC1815, Package_TO_SOT_THT:TO-92_Inline, symbol Transistor_BJT:2SC1815
- added Q3: TP29B/2SD880, Package_TO_SOT_THT:TO-92_Inline, symbol Transistor_BJT:2SC1815
- added R101: NOTE 8, symbol Device:R_US
- added R16, R36, R4: 1K, symbol Device:R_US
- added R17: 2.7K, symbol Device:R_US
- added R19: 15K, symbol Device:R_US
- added R2: 1.5K, symbol Device:R_US
- added R26, R52, R53: NOTE 2, symbol Device:R_US
- added R27: 500, symbol Device:R_Potentiometer_US
- added R3: 10K, symbol Device:R_US
- added R34: 47K, symbol Device:R_US
- added R45: 3.3K, symbol Device:R_US
- added R50: 1M, symbol Device:R_US
- added unit 1 of RP4
- added unit 2 of U20
- added U29: 74LS74_U29, symbol Commodore_64:74LS74_U29
- added U30: 74LS193_U30, symbol Commodore_64:74LS193_U30
- added U31: 74LS629N, symbol Commodore_64:74LS629N_U31
- added U32: MC4044_U32, symbol Commodore_64:MC4044_U32
- added unit 4 of U8
- added Y1: NOTE 2, symbol Device:Crystal_GND2
- U8: value 7406N -> 7406
- gave numbers to parts that had none: 1
- renumbered JP99 to E1
Connections:
- net +5V: now also C39.2, R34.1, R36.1, R45.2, R50.1, RP4.1, RP4.1, U20.10 (RST_{2}), U20.14 (VCC)
- net +9V: now also C18.2, Q1.2 (C), Q3.2 (C), R2.1
- net CAEC: now also U7.5 (AEC)
- net CASS RD: now also CN3.4 (RD), CN3.D (RD)
- net DOT_CLOCK: now also C36.2, FB17.2
- net GND: now also C105.1, C107.2, C108.2, C24.2, C36.1, C39.1, C56.1, C68.1, C74.1, C82.1, C83.1, C84.1, CR2.2 (A), E1., Q2.1 (E), R3.2, R52.2, U29.1 (~{R_{1}}), U29.2 (D_{1}), U29.3 (C_{1}), U29.7 (GND), U30.14 (CLR), U30.8 (GND), U31.11 (EN_{2}), U31.14 (RNG_{2}), U31.3 (RNG_{1}), U31.6 (EN_{1}), U31.8 (GND), U31.9 (GND), U32.7, Y1.2
- net ~{CHAREN}: now also U7.27 (P2), RP4.2
- net ~{HIRAM}: now also U7.28 (P1), RP4.3
- net ~{LORAM}: now also U7.29 (P0), R45.1
- net ~{RESET}: now also R36.2, U8.8
- net ɸ0: now also U7.1 (ɸ0), U32.3
- net ɸCOLOR: now also FB16.2, U30.5 (CNT_{UP})
- net CASS MOTOR: now reaches U7.24 (P5)
- net CASS MOTOR: now also CN3.3 (MOTOR), CN3.C (MOTOR), FB2.1, R4.1
- net CASS SENSE: now reaches U7.25 (P4)
- net CASS SENSE: now also CN3.6 (SENSE), CN3.F (SENSE)
- net CASS WRT: now reaches U7.26 (P3)
- net CASS WRT: now also CN3.5 (WRT), CN3.E (WRT), FB1.1, FB1.2
- new net: C86.2, R101.2, U31.4 (CX1_{1})
- new net: E1., U29.4 (~{PRE_{1}}), U30.1 (B), U30.10 (C)
- new net: C18.1, CR2.1 (K), Q1.3 (B), Q2.2 (C), R2.2
- new net: Q2.3 (B), R3.1, R4.2
- new net: R19.1, U32.10, U32.5 (VCC)
- new net: U32.11, U32.2
- new net: U32.13, U32.4
- new net: U20.9 (OUT_{2}), U8.9
- new net: C83.2, U30.11 (~{LOAD}), U30.12 (~{CO})
- new net: U29.11 (C_{2}), U30.6 (QC)
- new net: U29.5 (Q_{1}), U30.9 (D)
- new net: C85.1, R17.1
- new net: R16.2, R17.2, U31.2 (FC_{1}), U32.8
- new net: C85.2, Q7.3 (B), R19.2
- new net: C70.1, U31.13 (CX2_{2})
- new net: C70.2, Y1.3
- new net: FB17.1, U31.7 (Y_{1})
- new net: FB16.1, U31.10 (Y_{2})
- new net: U29.12 (D_{2}), U29.8 (~{Q_{2}})
- new net: U29.9 (Q_{2}), U32.1
- new net: C24.1, R34.2, U20.12 (THR_{2}), U20.13 (DIS_{2})
- new net: FB2.2, Q3.1 (E)
- new net: C107.1, R26.2, U31.15 (VCC)
- new net: C82.2, U29.14 (VCC)
- new net: Q7.1 (E), U32.9
- new net: C108.1, R27.2, U31.1 (FC_{2})
- new net: U31.12 (CX2_{2}), Y1.1
- new net: Q1.1 (E), Q3.3 (B)
- new net: C86.1, U31.5 (CX2_{1})
- new net: R27.1, R52.1
- new net: R27.3, R53.2
- new net: C105.2, R50.2, U20.8 (TRIG_{2})
- new net: CN3.1 (GND), CN3.A (GND)
- new net: CN3.2 (+5V), CN3.B (+5V)
- new net VCC: C56.2, C68.2, C74.2, C84.2, E1., Q7.2 (C), R101.1, R16.1, R26.1, R53.1, U29.10 (~{PRE_{2}}), U29.13 (~{R_{2}}), U30.15 (A), U30.16 (VCC), U30.4 (CNT_{DN}), U31.16 (VCC), U32.14
- no-connect marks 7 -> 12
Other:
- note added: "(14.31818 MHz - NTSC) (17.734472 MHz - PAL)"
- note added: "(6-PIN MALE EDGE)"
- note added: "JUMPER SELECT"
- note added: "U32 - MC4044"
