File: Apple/Apple II/Apple II - Memory Address Pt 1 of 2 (Rev 0,1).kicad_sch (KiCad schematic)
At the start: 0 parts

Commit message: Completed Apple II -  Memory Address Pt 1 of 2 (Rev 0,1)
Parts:
- added A2: 74LS00, symbol Apple II:A2_74LS00
- added C11: 74LS04, symbol Apple II:C11_74LS04
- added C14: 74LS32, symbol Apple II:C14_74LS32
- added D2: 74LS20, symbol Apple II:D2_74LS20
- added H1: 74LS08, symbol Apple II:H1_74LS08
- added N1 (x2): 1, symbol Apple II:NOTE_NUMBER
- added N2 (x2): 2, symbol Apple II:NOTE_NUMBER
- added U?: J1_74LS257, symbol Apple II:J1_74LS257
- added U?: F2_74LS139, symbol Apple II:F2_74LS139
- added U?: C12_74LS257, symbol Apple II:C12_74LS257
- added U?: D1_JUMPER_BLOCK, symbol Apple II:D1_JUMPER_BLOCK
- added U?: C1_74LS153, symbol Apple II:C1_74LS153
- added U?: E1_JUMPER_BLOCK, symbol Apple II:E1_JUMPER_BLOCK
- added U?: F1_JUMPER_BLOCK, symbol Apple II:F1_JUMPER_BLOCK
- added U?: E2_74LS139, symbol Apple II:E2_74LS139
Connections:
- new net: H1.8, U?.11 (0C)
- new net: U?.12 (ZC), U?.13 (2B), U?.13 (2B), U?.3 (1B)
- new net: U?.2 (0A), U?.6 (0A), U?.9 (ZD)
- new net: U?.3 (1B), U?.4 (ZA)
- new net: H1.11, U?.5 (0B)
- new net: U?.14 (2A), U?.2 (1A), U?.7 (ZB)
- new net: U?.14 (2A), U?.2 (1A), U?.9 (ZD)
- new net: H1.2, U?.10 (~{2Y2}), U?.8
- new net: H1.1, U?.11 (~{2Y1}), U?.9
- new net: U?.1 (~{1G}), U?.10, U?.12 (~{2Y0})
- new net: U?.10, U?.4 (~{1Y0})
- new net: U?.5 (~{1Y1}), U?.9
- new net: U?.6 (~{1Y2}), U?.8
- new net: A2.5, D2.8
- new net: D2.10, U?.13
- new net: D2.12, U?.14
- new net: D2.9, U?.12
- new net: U?.12 (ZC), U?.5 (1A)
- new net: U?.1, U?.1, U?.4 (~{1Y0})
- new net: U?.2, U?.2, U?.5 (~{1Y1})
- new net: U?.3, U?.3, U?.6 (~{1Y2})
- new net: U?.4, U?.4, U?.7 (~{1Y3})
- new net: U?.12 (~{2Y0}), U?.5, U?.5
- new net: U?.11 (~{2Y1}), U?.6, U?.6
- new net: U?.10 (~{2Y2}), U?.7, U?.7
- new net: U?.10, U?.7 (ZA), U?.8, U?.9
- new net: C14.2, H1.3
- new net: C14.3, U?.15 (~{2G})
- new net AD12_{14}: U?.3 (1A), U?.3 (3A)
- new net AD13_{15}: C14.1, U?.4 (2A), U?.6 (1B)
- new net AD14_{16}: U?.10 (1C)
- new net AD15_{17}: U?.13 (1D)
- new net AX: U?.14 (S0)
- new net Earth: U?.1 (~{EA}), U?.11 (0C), U?.14 (0D), U?.15 (~{2G}), U?.15 (~{E}), U?.15 (~{E})
- new net HBL: U?.14 (0D)
- new net HIRES: H1.10, H1.12, U?.1 (S)
- new net PAGE 2: C11.1, H1.9
- new net ROW C: U?.14
- new net ROW C ~{CAS}: U?.14
- new net ROW D: U?.13
- new net ROW D ~{CAS}: U?.13
- new net ROW E: U?.12
- new net ROW E ~{CAS}: U?.12
- new net R/W_{18}: A2.4
- new net VC: H1.13, U?.13 (1D)
- new net ~{CAS}: U?.1, U?.1 (~{1G}), U?.2, U?.3, U?.4, U?.5, U?.6, U?.7
- new net ~{KBD}: D2.13
- new net ~{PAGE 2}: C11.2, U?.10 (1C)
- new net ~{RAMSEL}: A2.6
- new net ɸ0_{40}: U?.1 (S), U?.2 (S1)
- no-connect marks 0 -> 1
Other:
- note added: "CIRCUIT FOR REV. 0"
- note added: "CIRCUIT FOR REV. 1"
- note added: "FROM CLOCK GENERATOR"
- note added: "FROM H1_{3}"
- note added: "FROM MICROPROCESSOR"
- note added: "FROM ON- BOARD I/O"
- note added: "FROM VIDEO ADDRESS GENERATOR"
- note added: "FROM VIDEO GENERATOR PART 1"
- note added: "FROM VIDEO GENERATOR PT 2"
- note added: "TO E2_{15}"
- note added: "TO ON- BOARD I/O"
- note added: "TO PART 2"
- note added: "TO RAM"
- title: (none) -> Apple II - Memory Address Part 1
