File: Apple/Apple II/Apple II - Peripheral IO (All Revisions).kicad_sch (KiCad schematic)
At the start: 0 parts

Commit message: Finished Apple II - Sheet 11 - Peripheral I/O (all revisions)
Parts:
- added CN?: IO_CONN_DETAIL, symbol Apple II:IO_CONN_DETAIL
- added H12: 74LS138, symbol Apple II:H12_74LS138
- added H2: 74LS138, symbol Apple II:H2_74LS138
- added JP10: USER 1 JUMPER, symbol Jumper:Jumper_2_Open
- added JP7: 7, symbol Jumper:SolderJumper_2_Open
- added JP8: 8, symbol Jumper:SolderJumper_2_Open
- added RA01: 1K, Resistor_THT:R_Array_SIP9, symbol Apple II:R_Network08_US_Split
- added S0: 0, symbol Apple II:IO_SLOT
- added S1: 1, symbol Apple II:IO_SLOT
- added S2: 2, symbol Apple II:IO_SLOT
- added S3: 3, symbol Apple II:IO_SLOT
- added S4: 4, symbol Apple II:IO_SLOT
- added S5: 5, symbol Apple II:IO_SLOT
- added S6: 6, symbol Apple II:IO_SLOT
- added S7: 7, symbol Apple II:IO_SLOT
Connections:
- new net: JP8.1 (A), S7.23 (INT_{OUT})
- new net: JP7.1 (A), S7.24 (DMA_{OUT})
- new net: S6.24 (DMA_{OUT}), S7.27 (DMA_{IN})
- new net: S6.23 (INT_{OUT}), S7.28 (INT_{IN})
- new net: S5.23 (INT_{OUT}), S6.28 (INT_{IN})
- new net: S5.24 (DMA_{OUT}), S6.27 (DMA_{IN})
- new net: S4.24 (DMA_{OUT}), S5.27 (DMA_{IN})
- new net: S4.23 (INT_{OUT}), S5.28 (INT_{IN})
- new net: S2.23 (INT_{OUT}), S3.28 (INT_{IN})
- new net: S2.24 (DMA_{OUT}), S3.27 (DMA_{IN})
- new net: S1.24 (DMA_{OUT}), S2.27 (DMA_{IN})
- new net: S1.23 (INT_{OUT}), S2.28 (INT_{IN})
- new net: S3.24 (DMA_{OUT}), S4.27 (DMA_{IN})
- new net: S3.23 (INT_{OUT}), S4.28 (INT_{IN})
- new net: S0.23 (INT_{OUT}), S1.28 (INT_{IN})
- new net: S0.24 (DMA_{OUT}), S1.27 (DMA_{IN})
- new net +12V: CN?.50 (+12V)
- new net +5V: CN?.25 (+5V), RA01.1 (R1.1)
- new net -12V: CN?.33 (-12V)
- new net -5V: CN?.34 (-5V)
- new net 7M_{36}: CN?.36 (7M)
- new net AD0_{2}: CN?.2 (AD0)
- new net AD10_{12}: CN?.12 (AD10), H12.3 (A2)
- new net AD11_{13}: CN?.13 (AD11)
- new net AD12_{14}: CN?.14 (AD12)
- new net AD13_{15}: CN?.15 (AD13)
- new net AD14_{16}: CN?.16 (AD14)
- new net AD15_{17}: CN?.17 (AD15)
- new net AD1_{3}: CN?.3 (AD1)
- new net AD2_{4}: CN?.4 (AD2)
- new net AD3_{5}: CN?.5 (AD3)
- new net AD4_{6}: CN?.6 (AD4), H2.1 (A0)
- new net AD5_{7}: CN?.7 (AD5), H2.2 (A1)
- new net AD6_{8}: CN?.8 (AD6), H2.3 (A2)
- new net AD7_{9}: CN?.9 (AD7), H2.6 (E3)
- new net AD8_{10}: CN?.10 (AD8), H12.1 (A0)
- new net AD9_{11}: CN?.11 (AD9), H12.2 (A1)
- new net B8_{2}: JP8.2 (B)
- new net COLOR_REF_{35}: CN?.35 (COLOR_REF)
- new net D0_{49}: CN?.49 (D0)
- new net D1_{48}: CN?.48 (D1)
- new net D2_{47}: CN?.47 (D2)
- new net D3_{46}: CN?.46 (D3)
- new net D4_{45}: CN?.45 (D4)
- new net D5_{44}: CN?.44 (D5)
- new net D6_{43}: CN?.43 (D6)
- new net D7_{42}: CN?.42 (D7)
- new net DMA_IN_{27}: CN?.27 (DMA_IN)
- new net DMA_OUT_{24}: CN?.24 (DMA_OUT)
- new net Earth: CN?.26 (GND)
- new net F12_{15}: H12.4 (~{E1}), H12.5 (~{E2})
- new net H12_{15}: H12.15 (~{Z0}), H2.4 (~{E1})
- new net INT_IN_{28}: CN?.28 (INT_IN)
- new net INT_OUT_{23}: CN?.23 (INT_OUT)
- new net M_{14}: JP7.2 (B)
- new net Q3_{37}: CN?.37 (Q3)
- new net RDY_{21}: CN?.21 (RDY)
- new net R/W_{18}: CN?.18 (R/W)
- new net SYNC_{19}: CN?.19 (SYNC)
- new net USER1_{39}: CN?.39 (USER1), H12.6 (E3), JP10.1 (A), JP10.2 (B), RA01.8 (R7.2)
- new net ~{DEV_SEL}_{41}: CN?.41 (~{DEV_SEL}), H2.10 (~{Z5}), H2.11 (~{Z4}), H2.12 (~{Z3}), H2.13 (~{Z2}), H2.14 (~{Z1}), H2.15 (~{Z0}), H2.7 (~{Z7}), H2.9 (~{Z6}), S0.41 (~{DEV_{SEL}}), S1.41 (~{DEV_{SEL}}), S2.41 (~{DEV_{SEL}}), S3.41 (~{DEV_{SEL}}), S4.41 (~{DEV_{SEL}}), S5.41 (~{DEV_{SEL}}), S6.41 (~{DEV_{SEL}}), S7.41 (~{DEV_{SEL}})
- new net ~{DMA}_{22}: CN?.22 (~{DMA})
- new net ~{INH}_{32}: CN?.32 (~{INH})
- new net ~{IRQ}_{30}: CN?.30 (~{IRQ})
- new net ~{I/O_SEL}_{1}: CN?.1 (~{I/O_SEL}), H12.10 (~{Z5}), H12.11 (~{Z4}), H12.12 (~{Z3}), H12.13 (~{Z2}), H12.14 (~{Z1}), H12.7 (~{Z7}), H12.9 (~{Z6}), S1.1 (~{I/O_{SEL}}), S2.1 (~{I/O_{SEL}}), S3.1 (~{I/O_{SEL}}), S4.1 (~{I/O_{SEL}}), S5.1 (~{I/O_{SEL}}), S6.1 (~{I/O_{SEL}}), S7.1 (~{I/O_{SEL}})
- new net ~{I/O_STB}_{20}: CN?.20 (~{I/O_STB})
- new net ~{NMI}_{29}: CN?.29 (~{NMI})
- new net ~{RESET}_{31}: CN?.31 (~{RESET})
- new net ɸ0_{40}: CN?.40 (ɸ0)
- new net ɸ1_{36}: H2.5 (~{E2})
- new net ɸ1_{38}: CN?.38 (ɸ1)
- no-connect marks 0 -> 3
Other:
- note added: "FROM CLOCK GENERATOR"
- note added: "FROM MICROPROCESOR"
- note added: "PERIPHERAL I/O CONNECTORS"
- note added: "TO ON- BOARD I/O"
- title: (none) -> Apple II - Peripheral I/O

Commit message: Fixed some missing notes on Apple II - Sheet 11 - Peripheral I/O (all revisions)
Parts:
- added N1 (x2): 1, symbol Apple II:NOTE_NUMBER
- added N2 (x2): 2, symbol Apple II:NOTE_NUMBER
Connections:
- net M_{14} is gone; now on net 14M: JP7.2 (B)
- net B8_{2}: now also JP8.1 (A), S7.23 (INT_{OUT})
- net 14M: now reaches JP7.1 (A), S7.24 (DMA_{OUT})
Other:
- note added: "FROM MICROPROCESSOR"
- note added: "FROM PERIPHERAL I/O CONNECTORS"
- note added: "FROM ROM"
- note added: "FROM VIDEO GENERATOR PT1"
- note added: "REV. 1, 7 AND RFI: SYNC AND COLOR REF CONNECT TO SLOT 7 ONLY; PINS 19 AND 35 FORM TWO BUSES FROM SLOT 0 TO SLOT 6. REV. 0: NO CONNECION TO SYNC OR COLOR REF; PINS 19 AND 35 FORM TWO BUSSES FROM SLOT 0 TO SLOT 7."
- note added: "REV. 7 AND RFI ONLY"
Changed lines of the file:
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@@
+    (stroke (width 0) (type solid) (color 0 0 0 0))
+  )
+  (polyline (pts (xy 264.795 36.83) (xy 263.525 36.83))
     (stroke (width 0) (type solid) (color 0 0 0 0))
   )
@@
     (stroke (width 0) (type default) (color 0 0 0 0))
   )
+  (polyline (pts (xy 35.56 246.38) (xy 34.29 246.38))
+    (stroke (width 0) (type solid) (color 0 0 0 0))
+  )
   (polyline (pts (xy 36.83 182.88) (xy 36.83 185.42))
     (stroke (width 0) (type solid) (color 0 0 0 0))
@@
     (stroke (width 0) (type default) (color 0 0 0 0))
   )
+  (polyline (pts (xy 263.525 29.21) (xy 263.525 31.75))
+    (stroke (width 0) (type solid) (color 0 0 0 0))
+  )
   (wire (pts (xy 80.01 87.63) (xy 80.01 104.14))
     (stroke (width 0) (type default) (color 0 0 0 0))
@@
     (stroke (width 0) (type default) (color 0 0 0 0))
   )
+  (polyline (pts (xy 35.56 228.6) (xy 35.56 238.76))
+    (stroke (width 0) (type solid) (color 0 0 0 0))
+  )
   (wire (pts (xy 279.4 119.38) (xy 276.86 119.38))
     (stroke (width 0) (type default) (color 0 0 0 0))
@@
     (stroke (width 0) (type solid) (color 0 0 0 0))
   )
+  (polyline (pts (xy 38.1 220.98) (xy 36.83 220.98))
+    (stroke (width 0) (type solid) (color 0 0 0 0))
+  )
   (wire (pts (xy 184.15 186.69) (xy 184.15 176.53))
     (stroke (width 0) (type default) (color 0 0 0 0))
   )
+  (polyline (pts (xy 264.795 39.37) (xy 263.525 39.37))
+    (stroke (width 0) (type solid) (color 0 0 0 0))
+  )
   (wire (pts (xy 163.83 30.48) (xy 46.99 30.48))
     (stroke (width 0) (type default) (color 0 0 0 0))
@@
     (stroke (width 0) (type default) (color 0 0 0 0))
   )
+  (polyline (pts (xy 288.29 25.4) (xy 288.29 41.91))
+    (stroke (width 0) (type default) (color 0 0 0 0))
+  )
   (polyline (pts (xy 39.37 64.77) (xy 38.1 64.77))
     (stroke (width 0) (type solid) (color 0 0 0 0))
@@
     (stroke (width 0) (type default) (color 0 0 0 0))
   )
+  (polyline (pts (xy 38.1 223.52) (xy 36.83 223.52))
+    (stroke (width 0) (type solid) (color 0 0 0 0))
+  )
   (wire (pts (xy 327.66 93.98) (xy 327.66 95.25))
     (stroke (width 0) (type default) (color 0 0 0 0))
@@
     (stroke (width 0) (type default) (color 0 0 0 0))
   )
+  (polyline (pts (xy 264.795 29.21) (xy 263.525 29.21))
+    (stroke (width 0) (type solid) (color 0 0 0 0))
+  )
   (wire (pts (xy 177.8 237.49) (xy 46.99 237.49))
     (stroke (width 0) (type default) (color 0 0 0 0))
@@
     (stroke (width 0) (type default) (color 0 0 0 0))
   )
+  (polyline (pts (xy 264.795 31.75) (xy 263.525 31.75))
+    (stroke (width 0) (type solid) (color 0 0 0 0))
+  )
   (wire (pts (xy 184.15 92.71) (xy 171.45 92.71))
     (stroke (width 0) (type default) (color 0 0 0 0))
@@
     (stroke (width 0) (type default) (color 0 0 0 0))
   )
+  (polyline (pts (xy 288.29 25.4) (xy 298.45 25.4))
+    (stroke (width 0) (type default) (color 0 0 0 0))
+  )
   (wire (pts (xy 255.27 85.09) (xy 255.27 90.17))
     (stroke (width 0) (type default) (color 0 0 0 0))
   )
+  (polyline (pts (xy 35.56 243.84) (xy 34.29 243.84))
+    (stroke (width 0) (type solid) (color 0 0 0 0))
+  )
   (wire (pts (xy 271.78 38.1) (xy 289.56 38.1))
     (stroke (width 0) (type default) (color 0 0 0 0))
@@
     (stroke (width 0) (type default) (color 0 0 0 0))
   )
+  (polyline (pts (xy 298.45 25.4) (xy 298.45 41.91))
+    (stroke (width 0) (type default) (color 0 0 0 0))
+  )
   (wire (pts (xy 46.99 34.29) (xy 156.21 34.29))
     (stroke (width 0) (type default) (color 0 0 0 0))
@@
     (stroke (width 0) (type default) (color 0 0 0 0))
   )
+  (polyline (pts (xy 263.525 36.83) (xy 263.525 39.37))
+    (stroke (width 0) (type solid) (color 0 0 0 0))
+  )
   (wire (pts (xy 96.52 129.54) (xy 93.98 129.54))
     (stroke (width 0) (type default) (color 0 0 0 0))
@@
     (stroke (width 0) (type default) (color 0 0 0 0))
   )
+  (polyline (pts (xy 34.29 243.84) (xy 34.29 246.38))
+    (stroke (width 0) (type solid) (color 0 0 0 0))
+  )
   (wire (pts (xy 279.4 129.54) (xy 276.86 129.54))
     (stroke (width 0) (type default) (color 0 0 0 0))
@@
     (stroke (width 0) (type default) (color 0 0 0 0))
   )
+  (polyline (pts (xy 36.83 238.76) (xy 35.56 238.76))
+    (stroke (width 0) (type solid) (color 0 0 0 0))
+  )
   (wire (pts (xy 166.37 186.69) (xy 166.37 179.07))
     (stroke (width 0) (type default) (color 0 0 0 0))
@@
     (stroke (width 0) (type default) (color 0 0 0 0))
   )
+  (polyline (pts (xy 36.83 220.98) (xy 36.83 223.52))
+    (stroke (width 0) (type solid) (color 0 0 0 0))
+  )
   (wire (pts (xy 95.25 184.15) (xy 130.81 184.15))
     (stroke (width 0) (type default) (color 0 0 0 0))
@@
     (stroke (width 0) (type default) (color 0 0 0 0))
   )
+  (polyline (pts (xy 298.45 41.91) (xy 288.29 41.91))
+    (stroke (width 0) (type default) (color 0 0 0 0))
+  )
+  (polyline (pts (xy 38.1 228.6) (xy 35.56 228.6))
+    (stroke (width 0) (type solid) (color 0 0 0 0))
+  )
   (polyline (pts (xy 64.135 109.22) (xy 59.69 109.22))
     (stroke (width 0) (type solid) (color 0 0 0 0))
@@
   (wire (pts (xy 189.23 245.11) (xy 195.58 245.11))
     (stroke (width 0) (type default) (color 0 0 0 0))
+  )
+  (text "FROM\nMICROPROCESSOR" (at 34.925 235.204 180)
+    (effects (font (size 0.96 0.96)) (justify right bottom))
+  )
+  (text "FROM CLOCK\nGENERATOR" (at 263.017 39.624 180)
+    (effects (font (size 0.96 0.96)) (justify right bottom))
+  )
+  (text "FROM\nROM" (at 36.322 223.774 180)
+    (effects (font (size 0.96 0.96)) (justify right bottom))
+  )
+  (text "REV. 1, 7 AND RFI: SYNC AND COLOR REF CONNECT TO SLOT\n7 ONLY; PINS 19 AND 35 FORM TWO BUSES FROM SLOT 0\nTO SLOT 6. REV. 0: NO CONNECION TO SYNC OR COLOR REF; PINS\n19 AND 35 FORM TWO BUSSES FROM SLOT 0 TO SLOT 7."
+    (at 303.53 241.935 0)
+    (effects (font (size 1.27 1.27)) (justify left bottom))
   )
   (text "FROM CLOCK\nGENERATOR" (at 37.592 67.564 180)
     (effects (font (size 0.96 0.96)) (justify right bottom))
   )
+  (text "FROM PERIPHERAL\nI/O CONNECTORS" (at 33.782 246.634 180)
+    (effects (font (size 0.96 0.96)) (justify right bottom))
+  )
   (text "TO ON-\nBOARD I/O" (at 36.322 185.674 180)
     (effects (font (size 0.96 0.96)) (justify right bottom))
   )
+  (text "REV. 7 AND RFI ONLY" (at 303.53 232.41 0)
+    (effects (font (size 1.27 1.27)) (justify left bottom))
+  )
   (text "FROM\nMICROPROCESOR" (at 37.465 38.1 180)
     (effects (font (size 0.96 0.96)) (justify right bottom))
   )
+  (text "FROM VIDEO\nGENERATOR PT1" (at 263.017 32.004 180)
+    (effects (font (size 0.96 0.96)) (justify right bottom))
+  )
   (text "PERIPHERAL I/O CONNECTORS" (at 58.42 163.83 90)
     (effects (font (size 2.54 2.54)) (justify left bottom))
   )
+  (label "14M" (at 299.72 38.1 0)
+    (effects (font (size 1.27 1.27)) (justify left bottom))
+  )
+  (label "B8_{2}" (at 299.72 30.48 0)
+    (effects (font (size 1.27 1.27)) (justify left bottom))
+  )
   (label "~{DEV_SEL}_{41}" (at 262.89 104.14 90)
     (effects (font (size 1.27 1.27)) (justify left bottom))
@@
     )
   )
-  (global_label "M_{14}" (shape input) (at 271.78 38.1 180) (fields_autoplaced)
-    (effects (font (size 1.27 1.27)) (justify right))
-    (property "Intersheet References" "${INTERSHEET_REFS}" (id 0) (at 265.9802 38.0206 0)
+  (global_label "14M" (shape input) (at 271.78 38.1 180) (fields_autoplaced)
+    (effects (font (size 1.27 1.27)) (justify right))
+    (property "Intersheet References" "${INTERSHEET_REFS}" (id 0) (at 265.4964 38.0206 0)
       (effects (font (size 1.27 1.27)) (justify right) hide)
     )
@@
     (pin "9")
   )
+  (symbol (lib_id "Apple II:NOTE_NUMBER") (at 300.99 234.95 0) (unit 1)
+    (in_bom yes) (on_board yes)
+    (property "Reference" "N2" (id 0) (at 293.37 229.87 0)
+      (effects (font (size 1.27 1.27)) hide)
+    )
+    (property "Value" "2" (id 1) (at 300.99 234.95 0))
+    (property "Footprint" "" (id 2) (at 300.99 234.95 0)
+      (effects (font (size 1.27 1.27)) hide)
+    )
+    (property "Datasheet" "" (id 3) (at 300.99 234.95 0)
+      (effects (font (size 1.27 1.27)) hide)
+    )
+  )
   (symbol (lib_id "Apple II:IO_SLOT") (at 101.6 109.22 0) (unit 1)
     (in_bom yes) (on_board yes)
@@
     (pin "41")
   )
+  (symbol (lib_id "Apple II:NOTE_NUMBER") (at 300.99 24.13 0) (unit 1)
+    (in_bom yes) (on_board yes)
+    (property "Reference" "N1" (id 0) (at 293.37 19.05 0)
+      (effects (font (size 1.27 1.27)) hide)
+    )
+    (property "Value" "1" (id 1) (at 300.99 24.13 0))
+    (property "Footprint" "" (id 2) (at 300.99 24.13 0)
+      (effects (font (size 1.27 1.27)) hide)
+    )
+    (property "Datasheet" "" (id 3) (at 300.99 24.13 0)
+      (effects (font (size 1.27 1.27)) hide)
+    )
+  )
   (symbol (lib_id "Jumper:SolderJumper_2_Open") (at 293.37 38.1 0) (mirror y) (unit 1)
     (in_bom yes) (on_board yes)
@@
     (pin "1")
     (pin "2")
+  )
+  (symbol (lib_id "Apple II:NOTE_NUMBER") (at 300.99 231.14 0) (unit 1)
+    (in_bom yes) (on_board yes)
+    (property "Reference" "N1" (id 0) (at 293.37 226.06 0)
+      (effects (font (size 1.27 1.27)) hide)
+    )
+    (property "Value" "1" (id 1) (at 300.99 231.14 0))
+    (property "Footprint" "" (id 2) (at 300.99 231.14 0)
+      (effects (font (size 1.27 1.27)) hide)
+    )
+    (property "Datasheet" "" (id 3) (at 300.99 231.14 0)
+      (effects (font (size 1.27 1.27)) hide)
+    )
   )
   (symbol (lib_id "power:+5V") (at 373.38 93.98 270) (unit 1)
@@
     (pin "41")
   )
+  (symbol (lib_id "Apple II:NOTE_NUMBER") (at 325.12 128.27 0) (unit 1)
+    (in_bom yes) (on_board yes)
+    (property "Reference" "N2" (id 0) (at 317.5 123.19 0)
+      (effects (font (size 1.27 1.27)) hide)
+    )
+    (property "Value" "2" (id 1) (at 325.12 128.27 0))
+    (property "Footprint" "" (id 2) (at 325.12 128.27 0)
+      (effects (font (size 1.27 1.27)) hide)
+    )
+    (property "Datasheet" "" (id 3) (at 325.12 128.27 0)
+      (effects (font (size 1.27 1.27)) hide)
+    )
+  )
 )
