File: Apple/Apple II/Apple II - Memory Address Pt 1 of 2 (Rev 7,RFI).kicad_sch (KiCad schematic)
At the start: 0 parts

Commit message: Finished Apple II - Sheet 5 - Memory Address Pt 1 of 2 (Rev 7,RFI)
Parts:
- added A2: 74LS00, symbol Apple II:A2_74LS00
- added C11: 74LS04, symbol Apple II:C11_74LS04
- added D2: 74LS20, symbol Apple II:D2_74LS20
- added H1: 74LS08, symbol Apple II:H1_74LS08
- added R31, R32: 1K, symbol Device:R_US
- added U?: J1_74LS257, symbol Apple II:J1_74LS257
- added U?: F2_74LS139, symbol Apple II:F2_74LS139
- added U?: C1_74LS153, symbol Apple II:C1_74LS153
- added U?: C12_74LS257, symbol Apple II:C12_74LS257
Connections:
- new net: H1.8, U?.11 (0C)
- new net: U?.12 (ZC), U?.13 (2B), U?.3 (1B)
- new net: U?.14 (2A), U?.2 (1A), U?.9 (ZD)
- new net: D2.9, U?.10 (~{2Y2})
- new net: D2.10, U?.11 (~{2Y1})
- new net: D2.12, U?.12 (~{2Y0})
- new net: A2.5, D2.8
- new net: U?.12 (ZC), U?.5 (1A)
- new net: U?.6 (0A), U?.9 (ZD)
- new net +5V: R32.1
- new net AD12_{14}: U?.3 (3A)
- new net AD13_{15}: U?.4 (2A)
- new net AD14_{16}: U?.10 (1C)
- new net AD15_{17}: U?.13 (1D)
- new net AX: U?.14 (S0)
- new net Earth: R31.2, U?.1 (~{EA}), U?.11 (0C), U?.14 (0D), U?.15 (~{E}), U?.15 (~{E})
- new net HBL: U?.14 (0D)
- new net HIRES: H1.10, U?.1 (S)
- new net PAGE 2: C11.1, H1.9
- new net ROW C RA6: R31.1, R32.2, U?.7 (ZA)
- new net ROW C ~{CAS}: U?.4 (~{1Y0})
- new net ROW D ~{CAS}: U?.5 (~{1Y1})
- new net ROW E ~{CAS}: U?.6 (~{1Y2})
- new net R/W_{18}: A2.4
- new net VC: U?.13 (1D)
- new net ~{CAS}: U?.1 (~{1G})
- new net ~{KBD}: D2.13
- new net ~{PAGE 2}: C11.2, U?.10 (1C)
- new net ~{RAMSEL}: A2.6
- new net ɸ0_{40}: U?.1 (S), U?.2 (S1)
Other:
- note added: "FROM CLOCK GENERATOR"
- note added: "FROM MICROPROCESSOR"
- note added: "FROM ON- BOARD I/O"
- note added: "FROM VIDEO ADDRESS GENERATOR"
- note added: "FROM VIDEO GENERATOR PART 1"
- note added: "FROM VIDEO GENERATOR PT 2"
- note added: "TO ON- BOARD I/O"
- note added: "TO PART 2"
- note added: "TO RAM"
- title: (none) -> Apple II - Memory Address Part 1
