File: Apple/Apple II/Apple II - Memory Address Pt 2 of 2 (All Revisions).kicad_sch (KiCad schematic)
At the start: 0 parts

Commit message: Finished Apple II - Sheet 6 - Memory Address Pt 2 of 2 (All Revisions)
Parts:
- added C11: 74LS04, symbol Apple II:C11_74LS04
- added E12: E12_74LS153, symbol Apple II:E12_74LS153
- added E13: E13_74LS153, symbol Apple II:E13_74LS153
- added N1, N?: 1, symbol Apple II:NOTE_NUMBER
- added RA02, RA03: 1K, Resistor_THT:R_Array_SIP9, symbol Apple II:R_Network08_US_Split
- added U?: E11_74LS153, symbol Apple II:E11_74LS153
- added U?: E14_74LS283, symbol Apple II:E14_74LS283
- added U?: C12_74LS257, symbol Apple II:C12_74LS257
Connections:
- new net: U?.10 (0B), U?.7 (ZB)
- new net: U?.4 (ZA), U?.6 (0A)
- new net: C11.6, U?.12 (A3), U?.15 (B2)
- new net +5V: RA02.1 (R1.1), RA02.1 (R1.1), RA02.1 (R1.1), RA02.1 (R1.1), RA02.1 (R1.1), RA02.1 (R1.1)
- new net AD0_{2}: E13.3 (3A)
- new net AD10_{12}: U?.5 (1A)
- new net AD11_{13}: U?.11 (1B)
- new net AD1_{3}: E13.13 (3B)
- new net AD2_{4}: E12.3 (3A)
- new net AD3_{5}: E12.13 (3B)
- new net AD4_{6}: E12.5 (1A)
- new net AD5_{7}: E13.5 (1A)
- new net AD6_{8}: E13.11 (1B)
- new net AD7_{9}: U?.3 (3A)
- new net AD8_{10}: U?.13 (3B)
- new net AD9_{11}: E12.11 (1B)
- new net AX: E12.2 (S1), E13.2 (S1), U?.2 (S1)
- new net Earth: E12.1 (~{EA}), E12.15 (~{EB}), E13.1 (~{EA}), E13.15 (~{EB}), RA03.1 (R1.1), RA03.1 (R1.1), RA03.1 (R1.1), RA03.1 (R1.1), RA03.1 (R1.1), RA03.1 (R1.1), U?.1 (~{EA}), U?.15 (~{EB}), U?.15 (~{E})
- new net H0: E13.4 (2A)
- new net H1: E13.12 (2B)
- new net H2: E12.4 (2A)
- new net H3: U?.5 (A0)
- new net H4: U?.3 (A1)
- new net H5: C11.5
- new net HIRES: U?.1 (S)
- new net PAGE 2: U?.5 (0B)
- new net RA0: RA02.7 (R6.2), RA03.7 (R6.2), U?.7 (ZA)
- new net RA1: E12.7 (ZA), RA02.5 (R4.2), RA03.5 (R4.2)
- new net RA2: E13.7 (ZA), RA02.3 (R2.2), RA03.3 (R2.2)
- new net RA3: RA02.8 (R7.2), RA03.8 (R7.2), U?.9 (ZB)
- new net RA4: E12.9 (ZB), RA02.6 (R5.2), RA03.6 (R5.2)
- new net RA5: E13.9 (ZB), RA02.4 (R3.2), RA03.4 (R3.2)
- new net SOFT 5: U?.6 (B0)
- new net V0: U?.4 (2A)
- new net V1: U?.12 (2B)
- new net V2: E12.10 (0B)
- new net V3: U?.14 (A2), U?.7 (C_{IN})
- new net V4: U?.11 (B3), U?.2 (B1)
- new net VA: U?.3 (1A)
- new net VB: U?.6 (1B)
- new net ~{PAGE 2}: U?.2 (0A)
- new net ɸ0_{40}: E12.14 (S0), E13.14 (S0), U?.14 (S0)
- new net ∑0: E12.12 (2B), U?.4 (∑0)
- new net ∑1: E12.6 (0A), U?.1 (∑1)
- new net ∑2: E13.6 (0A), U?.13 (∑2)
- new net ∑3: E13.10 (0B), U?.10 (∑3)
- no-connect marks 0 -> 1
Other:
- note added: "1K"
- note added: "AD SIGNALS ARE FROM MICROPROCESSOR. H AND V SIGNALS ARE FROM VIDEO ADDRESS GENERATOR."
- note added: "FROM CLOCK GENERATOR"
- note added: "FROM PART 1"
- note added: "FROM PERIPHERAL I/O"
- note added: "FROM VIDEO ADDRESS GENERATOR"
- note added: "FROM VIDEO GENERATOR PT 1"
- note added: "RA02"
- note added: "RA03"
- note added: "TO RAM"
- title: (none) -> Apple II - Memory Address Part 2
