File: Apple/Apple II/Apple II - RAM (All Revisions).kicad_sch (KiCad schematic)
At the start: 0 parts

Commit message: Finished Apple II - Sheet 7 - RAM (all revisions)
Parts:
- added C14: 74LS32, symbol Apple II:C14_74LS32
- added U?: 4116_RAM_ARRAY, symbol Apple II:4116_RAM_ARRAY
- added U?: 4116_POWER, symbol Apple II:4116_POWER
- added U?: B5_74LS174, symbol Apple II:B5_74LS174
- added U?: B8_74LS174, symbol Apple II:B8_74LS174
Connections:
- new net: U?.11 (D3), U?.14 (D_{O}) (x2)
- new net: U?.13 (D4), U?.14 (D_{O}) (x2)
- new net: U?.14 (D_{O}), U?.4 (D1) (x2)
- new net: U?.14 (D_{O}), U?.6 (D2) (x2)
- new net: C14.11, U?.3 (~{WR})
- new net +12V: U?.8 (V_{DD})
- new net +5V: U?.9 (V_{CC})
- new net -5V: U?.1 (V_{BB})
- new net D0_{49}: U?.2 (D_{I})
- new net D1_{48}: U?.2 (D_{I})
- new net D2_{47}: U?.2 (D_{I})
- new net D3_{46: U?.2 (D_{I})
- new net D4_{45}: U?.2 (D_{I})
- new net D5_{44}: U?.2 (D_{I})
- new net D6_{43}: U?.2 (D_{I})
- new net D7_{42}: U?.2 (D_{I})
- new net DL0: U?.10 (Q3)
- new net DL1: U?.12 (Q4)
- new net DL2: U?.5 (Q1)
- new net DL3: U?.7 (Q2)
- new net DL4: U?.10 (Q3)
- new net DL5: U?.12 (Q4)
- new net DL6: U?.5 (Q1)
- new net DL7: U?.7 (Q2)
- new net Earth: U?.16 (GND)
- new net RA0: U?.10 (A0)
- new net RA1: U?.11 (A1)
- new net RA2: U?.12 (A2)
- new net RA3: U?.7 (A3)
- new net RA4: U?.6 (A4)
- new net RA5: U?.5 (A5)
- new net ROW C RA6: U?.13 (A6)
- new net ROW C ~{CAS}: U?.15 (~{CAS})
- new net ROW D RA6: U?.13 (A6)
- new net ROW D ~{CAS}: U?.15 (~{CAS})
- new net ROW E RA6: U?.13 (A6)
- new net ROW E ~{CAS}: U?.15 (~{CAS})
- new net R/W_{18}: C14.13
- new net SOFT 5: U?.1 (~{CLR}), U?.1 (~{CLR})
- new net ~{RAS}: U?.4 (~{RAS}), U?.9 (Cp), U?.9 (Cp)
- new net ɸ1_{38}: C14.12
Other:
- note added: "FROM CLOCK GENERATOR"
- note added: "FROM MEMORY ADDRESS PT 1"
- note added: "FROM MEMORY ADDRESS PT 2"
- note added: "FROM MICROPROCESSOR"
- note added: "TO PERIPHERAL I/O AND VIDEO GENERATOR"
- title: (none) -> Apple II - RAM
