File: Apple/Apple II/Apple II - Microprocessor (Rev RFI).kicad_sch (KiCad schematic)
At the start: 0 parts

Commit message: Finished Apple II - Sheet 9 - Microprocessor (Rev RFI)
Parts:
- added B?: 74LS08, symbol Apple II:B11_74LS08
- added C?: 74LS04, symbol Apple II:C11_74LS04
- added C?: 74LS32, symbol Apple II:C14_74LS32
- added N? (x2): 1, symbol Apple II:NOTE_NUMBER
- added RA? (x5): 1K, Resistor_THT:R_Array_SIP9, symbol Apple II:R_Network08_US_Split
- added U? (x5): H3_8T97, symbol Apple II:H3_8T97
- added U? (x7): H4_8T97, symbol Apple II:H4_8T97
- added U? (x5): H5_8T97, symbol Apple II:H5_8T97
- added U?: H10_8304, symbol Apple II:H10_8304
- added U?: H8_6502, symbol Apple II:H8_6502
Connections:
- new net: C?.12, U?.1, U?.1, U?.1, U?.1, U?.1, U?.1, U?.1, U?.1, U?.1, U?.1, U?.1, U?.15, U?.15, U?.15, U?.15, U?.15, U?.15
- new net: U?.18 (A9), U?.2
- new net: U?.19 (A10), U?.9
- new net: U?.11, U?.20 (A11)
- new net: U?.13, U?.25 (A15)
- new net: U?.11, U?.9 (A0)
- new net: U?.11 (A2), U?.6
- new net: U?.13 (A4), U?.6
- new net: B?.3, U?.37 (ɸ0)
- new net: U?.13, U?.24 (A14)
- new net: U?.16 (A7), U?.6
- new net: U?.2, U?.23 (A13)
- new net: U?.2, U?.22 (A12)
- new net: C?.8, U?.11
- new net: U?.12, U?.26 (D7)
- new net: U?.13, U?.27 (D6)
- new net: U?.14, U?.28 (D5)
- new net: U?.15, U?.29 (D4)
- new net: U?.16, U?.30 (D3)
- new net: U?.17, U?.31 (D2)
- new net: U?.18, U?.32 (D1)
- new net: U?.19, U?.33 (D0)
- new net: U?.17 (A8), U?.4
- new net: U?.10 (A1), U?.4
- new net: U?.14 (A5), U?.9
- new net: U?.11, U?.15 (A6)
- new net: C?.10, U?.3 (ɸ1)
- new net: U?.13, U?.34 (R/W)
- new net: U?.12 (A3), U?.9
- new net +5V: RA?.1 (R1.1), RA?.1 (R1.1), RA?.1 (R1.1), RA?.1 (R1.1), RA?.1 (R1.1), U?.8 (V_{CC})
- new net AD0_{2}: U?.12
- new net AD10_{12}: U?.10
- new net AD11_{13}: U?.12
- new net AD12_{14}: U?.3
- new net AD13_{15}: U?.3
- new net AD14_{16}: U?.14
- new net AD15_{17}: U?.14
- new net AD1_{3}: U?.5
- new net AD2_{4}: U?.7
- new net AD3_{5}: U?.10
- new net AD4_{6}: U?.7
- new net AD5_{7}: U?.10
- new net AD6_{8}: U?.12
- new net AD7_{9}: U?.7
- new net AD8_{10}: U?.5
- new net AD9_{11}: U?.3
- new net D0_{49}: U?.1
- new net D1_{48}: U?.2
- new net D2_{47}: U?.3
- new net D3_{46}: U?.4
- new net D4_{45}: U?.5
- new net D5_{44}: U?.6
- new net D6_{43}: U?.7
- new net D7_{42}: U?.8
- new net Earth: U?.1 (V_{SS}), U?.21 (V_{SS}), U?.9 (~{E})
- new net RDY_{21}: RA?.5 (R4.2), U?.2 (RDY)
- new net R/W_{18}: C?.9, U?.14
- new net ~{DMA}_{22}: B?.1, C?.13, RA?.3 (R2.2)
- new net ~{IRQ}_{30}: RA?.4 (R3.2), U?.4 (~{IRQ})
- new net ~{NMI}_{29}: RA?.2 (R1.2), U?.6 (~{NMI})
- new net ~{RESET}_{31}: U?.40 (~{RES})
- new net ɸ0_{40}: B?.2
- no-connect marks 0 -> 2
Other:
- note added: "1K"
- note added: "8T97"
- note added: "FROM CLOCK GENERATOR"
- note added: "FROM KEYBOARD AND PERIPHERAL I/O"
- note added: "FROM PERIPHERAL I/O"
- note added: "MAY BE SUBSTITUTED WITH 74LS367 ON SOME BOARDS"
- note added: "RA01"
- note added: "SYSTEM ADDRESS BUS"
- note added: "SYSTEM DATA BUS"
- title: (none) -> Apple II - Microprocessor
