File: Apple/Apple II/Apple II - On-board IO Pt 1 of 2 (All Revisions).kicad_sch (KiCad schematic)
At the start: 0 parts

Commit message: Finished Apple II - Sheet 12 - On-Board I/O Pt 1 of 2 (all revisions)
Parts:
- added C10, C11, C12, C9: 0.1µF, symbol Device:C_Small
- added C5, C6, C7, C8: 0.022µF, symbol Device:C_Small
- added CN?: J14_GAME_IO_CONN, symbol Apple II:J14_GAME_IO_CONN
- added CR1: 1N914, symbol Device:D_Filled
- added F13: 74LS138, symbol Apple II:F13_74LS138
- added F14: 74LS259, symbol Apple II:F14_74LS259
- added H14: 74LS251, symbol Apple II:H14_74LS251
- added J13: 74LS74, symbol Apple II:J13_74LS74
- added J45: CASSETTE DATA OUT, symbol Connector:Conn_Coaxial
- added J98: CASSETTE DATA IN, symbol Connector:Conn_Coaxial
- added N1 (x2): 1, symbol Apple II:NOTE_NUMBER
- added N2, N?: 2, symbol Apple II:NOTE_NUMBER
- added Q4: MPSA13, symbol Apple II:Q4_MPSA13
- added R15: 1M, symbol Device:R_US
- added R16, R17, R19, R29, R30: 12K, symbol Device:R_US
- added R18, R20, R21, R22, R23: 100Ω, symbol Device:R_US
- added R24: 47K, symbol Device:R_US
- added R5: 27Ω, symbol Device:R_US
- added SPEAKER: 8Ω, symbol Device:Speaker
- added TP1: TestPoint, symbol Connector:TestPoint
- added U?: K13_LM741, symbol Apple II:K13_LM741
- added U?: H13_558_TIMER, symbol Apple II:H13_558_TIMER
Connections:
- new net: CN?.10 (PDL_{1}), R21.1
- new net: C5.1, R21.2, U?.15 (D)
- new net: Q4., R5.1
- new net: C12.2, R5.2, SPEAKER.2
- new net: H14.4 (D0), R29.1
- new net: R15.2, R29.2, U?.6
- new net: F13.10 (~{Z5}), F14.14 (~{E})
- new net: CN?.5 (~{STB}), F13.11 (~{Z4})
- new net: F13.12 (~{Z3}), J13.3 (CLK)
- new net: F13.13 (~{Z2}), J13.11 (CLK)
- new net: F13.7 (~{Z7}), U?.11 (TR_{C}), U?.14 (TR_{D}), U?.3 (TR_{A}), U?.6 (TR_{B})
- new net: F13.9 (~{Z6}), H14.7 (~{E})
- new net: J13.12 (D), J13.8 (~{Q}), R19.1
- new net: C7.1, R23.2, U?.7 (B)
- new net: CN?.15 (AN0), F14.9 (Z4), TP1.1
- new net: CR1.1 (K), Q4., R24.2
- new net: C11.2, R24.1
- new net: C8.1, R20.2, U?.2 (A)
- new net: J45.1 (In), R18.2, R19.2
- new net: CN?.6 (PDL_{0}), R20.1
- new net: CN?.4 (SW2), H14.1 (D3)
- new net: H14.12 (D7), U?.8 (Q_{B})
- new net: H14.13 (D6), U?.9 (Q_{C})
- new net: H14.14 (D5), U?.16 (Q_{D})
- new net: H14.15 (D4), U?.1 (Q_{A})
- new net: CN?.3 (SW1), H14.2 (D2)
- new net: CN?.2 (SW0), H14.3 (D1)
- new net: CN?.11 (PDL_{3}), R23.1
- new net: R17.1, R30.1, U?.2 (-)
- new net: R15.1, R16.2, U?.3 (+)
- new net: CN?.14 (AN1), F14.10 (Z5)
- new net: CN?.12 (AN3), F14.12 (Z7)
- new net: C6.1, R22.2, U?.10 (C)
- new net: C10.1, J98.1 (In)
- new net: C9.1, U?.4 (CV)
- new net: CN?.7 (PDL_{2}), R22.1
- new net: J13.2 (D), J13.6 (~{Q})
- new net: C11.1, J13.5 (Q)
- new net: C10.2, R30.2
- new net +5V: CN?.1 (+5V), SPEAKER.1, U?.13 (~{RES}), U?.5 (V_{CC}), U?.7
- new net -5V: U?.4
- new net AD0_{2}: F14.13 (D), H14.11 (A)
- new net AD1_{3}: F14.1 (A), H14.10 (B)
- new net AD2_{4}: F14.2 (B), H14.9 (C)
- new net AD3_{5}: F14.3 (C)
- new net AD4_{6}: F13.1 (A)
- new net AD5_{7}: F13.2 (B)
- new net AD6_{8}: F13.3 (C)
- new net AD7_{9}: F13.4 (~{E1})
- new net AN2: CN?.13 (AN2), F14.11 (Z6)
- new net D7_{42}: H14.5 (Y)
- new net Earth: C12.1, C5.2, C6.2, C7.2, C8.2, C9.2, CN?.6 (PDL_{0}), CR1.2 (A), J45.2 (Ext), J98.2 (Ext), Q4., R16.1, R17.2, R18.1, U?.12 (GND)
- new net H12_{15}: F13.5 (~{E2})
- new net HIRES MODE: F14.7 (Z3)
- new net MIX MODE: F14.5 (Z1)
- new net PAGE 2: F14.6 (Z2)
- new net SOFT 5: F14.15 (~{CLR}), J13.1 (~{CLR}), J13.10 (~{P}), J13.13 (~{CLR}), J13.4 (~{P})
- new net TEXT MODE: F14.4 (Z0)
- new net ~{CLR_STB}: F13.14 (~{Z1})
- new net ~{KBD}: F13.15 (~{Z0})
- new net ɸ0_{40}: F13.6 (E3)
- no-connect marks 0 -> 3
Other:
- note added: "FROM CLOCK GENERATOR"
- note added: "FROM MICROPROCESSOR"
- note added: "FROM PERIPHERAL I/O"
- note added: "ON REV. 0 AND SOME REV. 1 BOARDS, R15 IS 220K OR 470K AND R30 IS OMITTED."
- note added: "REV. 7 AND RFI ONLY"
- note added: "TO MEMORY ADDRESS"
- note added: "TO MICROPROCESSOR"
- note added: "TO PART 2"
- note added: "TO VIDEO GENERATOR PT 1"
- title: (none) -> Apple II - On-Board I/O Part 1
