File: Apple/Apple II/Apple II - On-board IO Pt 2 of 2 (All Revisions).kicad_sch (KiCad schematic)
At the start: 0 parts

Commit message: Finished Apple II - Sheet 13 - On-Board I/O Part 2
Parts:
- added A12: 74LS02, symbol Apple II:A12_74LS02
- added B10: 74LS74, symbol Apple II:B10_74LS74
- added C11: 74LS04, symbol Apple II:C11_74LS04
- added C4: 0.1µF, symbol Device:C_Small
- added N1 (x2): 1, symbol Apple II:NOTE_NUMBER
- added N2 (x2): 2, symbol Apple II:NOTE_NUMBER
- added Q5: 2N3904, Package_TO_SOT_THT:TO-92_Inline, symbol Transistor_BJT:2N3904
- added R14: 1K, symbol Device:R_US
- added R26: 2.2M, symbol Device:R_US
- added U?: A13_555, Package_SO:SOIC-8_3.9x4.9mm_P1.27mm, symbol Apple II:A13_555
- added U?: B7_74LS257, symbol Apple II:B7_74LS257
- added U?: A7_KEYBOARD_CONN, symbol Apple II:A7_KEYBOARD_CONN
- added U?: B6_74LS257, symbol Apple II:B6_74LS257
Connections:
- new net: Q5.2 (B), R14.2
- new net: C4.1, R26.1, U?.2 (TR), U?.6 (TH)
- new net: A12.3, R14.1, U?.3 (OUT)
- new net: B10.11 (CLK), U?.2 (STROBE)
- new net: A12.1, B10.13 (~{CLR})
- new net: B10.9 (Q), U?.5 (0B)
- new net: U?.11 (0C), U?.6 (B5)
- new net: U?.14 (0D), U?.5 (B6)
- new net: U?.2 (0A), U?.7 (B7)
- new net: A12.2, C11.4
- new net: U?.10 (B3), U?.2 (0A)
- new net: U?.11 (B4), U?.5 (0B)
- new net: U?.11 (0C), U?.12 (B1)
- new net: U?.13 (B2), U?.14 (0D)
- new net +5V: R26.2, U?.1 (+5V), U?.4 (~{R}), U?.8 (VCC)
- new net -12V: U?.15 (-12V)
- new net B10_{13}: C11.3
- new net D0_{49}: U?.12 (ZC)
- new net D1_{48}: U?.9 (ZD)
- new net D2_{47}: U?.4 (ZA)
- new net D3_{46}: U?.7 (ZB)
- new net D4_{45}: U?.9 (ZC)
- new net D5_{44}: U?.12 (ZD)
- new net D6_{43}: U?.4 (ZA)
- new net D7_{42}: U?.7 (ZB)
- new net DL0: U?.10 (1C)
- new net DL1: U?.13 (1D)
- new net DL2: U?.3 (1A)
- new net DL3: U?.6 (1B)
- new net DL4: U?.10 (1C)
- new net DL5: U?.13 (1D)
- new net DL6: U?.3 (1A)
- new net DL7: U?.6 (1B)
- new net Earth: C4.2, Q5.1 (E), U?.1 (GND), U?.8 (GND)
- new net SOFT 5: B10.10 (~{P}), B10.12 (D)
- new net ~{KBD}: U?.1 (S), U?.1 (S)
- new net ~{RAM_SEL}: U?.15 (~{E}), U?.15 (~{E})
- new net ~{RESET}_{31}: Q5.3 (C), U?.3 (~{RESET})
- no-connect marks 0 -> 2
Other:
- note added: "ALTERNATE CIRCUIT FOR REV. 0"
- note added: "B10_{12} IS OPEN ON REV. 0"
- note added: "DATA BUS"
- note added: "FROM MICROPROCESSOR"
- note added: "FROM PART 1"
- note added: "POWER ON RESET"
- title: (none) -> Apple II - On-Board I/O Part 2
