File: Apple/Apple II/Apple II - ROM (All Revisions).kicad_sch (KiCad schematic)
At the start: 6 parts

Commit message: Working on the Apple II Sheet 23
Connections:
- net at U?.20 (~{CS1}), U?.21 (~{CS3}): now also F12.9 (~{Z6}); no longer F12.10 (~{Z5})
- new net: F12.10 (~{Z5}), U?.20 (~{CS1}), U?.21 (~{CS3})
- new net: F12.11 (~{Z4}), U?.20 (~{CS1}), U?.21 (~{CS3})
- new net: F12.12 (~{Z3}), U?.20 (~{CS1}), U?.21 (~{CS3})
- new net: F12.13 (~{Z2}), U?.20 (~{CS1}), U?.21 (~{CS3})
- new net: F12.7 (~{Z7}), U?.20 (~{CS1}), U?.21 (~{CS3})

Commit message: More Apple II Power Supply work
Connections:
- net at U?.20 (~{CS1}), U?.21 (~{CS3}): now also F12.9 (~{Z6}); no longer F12.10 (~{Z5})
- new net: F12.10 (~{Z5}), U?.20 (~{CS1}), U?.21 (~{CS3})
- new net: F12.11 (~{Z4}), U?.20 (~{CS1}), U?.21 (~{CS3})
- new net: F12.12 (~{Z3}), U?.20 (~{CS1}), U?.21 (~{CS3})
- new net: F12.13 (~{Z2}), U?.20 (~{CS1}), U?.21 (~{CS3})
- new net: F12.7 (~{Z7}), U?.20 (~{CS1}), U?.21 (~{CS3})

Commit message: Apple II Complete!
All done!  Release to follow!
Connections:
- net at U?.20 (~{CS1}), U?.21 (~{CS3}): now also F12.9 (~{Z6}); no longer F12.10 (~{Z5})
- new net: F12.10 (~{Z5}), U?.20 (~{CS1}), U?.21 (~{CS3})
- new net: F12.11 (~{Z4}), U?.20 (~{CS1}), U?.21 (~{CS3})
- new net: F12.12 (~{Z3}), U?.20 (~{CS1}), U?.21 (~{CS3})
- new net: F12.13 (~{Z2}), U?.20 (~{CS1}), U?.21 (~{CS3})
- new net: F12.7 (~{Z7}), U?.20 (~{CS1}), U?.21 (~{CS3})
