File: Apple/Apple II/Apple II - Two-piece Keyboard.kicad_sch (KiCad schematic)
At the start: 0 parts

Commit message: Finished Apple II - Sheet 22 - Two-Piece Keyboard
Parts:
- added C1: 1µF, symbol Device:C_Polarized_Small
- added C2: 0.02µF, symbol Device:C_Small
- added C3, C4, C6, C7, C8: 0.1µF, symbol Device:C_Small
- added C5: 47pF, symbol Device:C_Small
- added D?: TPK_S54_POWER_INDICATOR, symbol Apple II:TPK_S54_POWER_INDICATOR
- added KBD?: TPK_TWO_PIECE_KEYBOARD, symbol Apple II:TPK_TWO_PIECE_KEYBOARD
- added KBDN10: 10, symbol Apple II:KBD_NOTE_J1_2PIN
- added KBDN10: 10, symbol Apple II:KBD_NOTE_P1
- added KBDN11: 11, symbol Apple II:KBD_NOTE_P1
- added KBDN11: 11, symbol Apple II:KBD_NOTE_J1_2PIN
- added KBDN12: 12, symbol Apple II:KBD_NOTE_J1_2PIN
- added KBDN12: 12, symbol Apple II:KBD_NOTE_P1
- added KBDN13: 13, symbol Apple II:KBD_NOTE_P1
- added KBDN13: 13, symbol Apple II:KBD_NOTE_J1_2PIN
- added KBDN14: 14, symbol Apple II:KBD_NOTE_P1
- added KBDN15: 15, symbol Apple II:KBD_NOTE_P1
- added KBDN15: 15, symbol Apple II:KBD_NOTE_J1_2PIN
- added KBDN16: 16, symbol Apple II:KBD_NOTE_P1
- added KBDN17: 17, symbol Apple II:KBD_NOTE_P1
- added KBDN18: 18, symbol Apple II:KBD_NOTE_P1
- added KBDN2: 2, symbol Apple II:KBD_NOTE_J1_1PIN
- added KBDN2: 2, symbol Apple II:KBD_NOTE_P1
- added KBDN21: 21, symbol Apple II:KBD_NOTE_P1
- added KBDN22: 22, symbol Apple II:KBD_NOTE_P1
- added KBDN23 (x3): 23, symbol Apple II:KBD_NOTE_P1
- added KBDN24: 24, symbol Apple II:KBD_NOTE_P1
- added KBDN3: 3, symbol Apple II:KBD_NOTE_P1
- added KBDN3: 3, symbol Apple II:KBD_NOTE_J1_1PIN
- added KBDN4: 4, symbol Apple II:KBD_NOTE_P1
- added KBDN5: 5, symbol Apple II:KBD_NOTE_J1_2PIN
- added KBDN5: 5, symbol Apple II:KBD_NOTE_P1
- added KBDN56: 56, symbol Apple II:KBD_NOTE_P1
- added KBDN6: 6, symbol Apple II:KBD_NOTE_P1
- added KBDN6: 6, symbol Apple II:KBD_NOTE_J1_2PIN
- added KBDN7: 7, symbol Apple II:KBD_NOTE_P1
- added KBDN7: 7, symbol Apple II:KBD_NOTE_J1_2PIN
- added KBDN8: 8, symbol Apple II:KBD_NOTE_J1_2PIN
- added KBDN8: 8, symbol Apple II:KBD_NOTE_P1
- added KBDN9, KBDN?: 9, symbol Apple II:TPK_TRIANGLE_NOTE
- added KBDN9: 9, symbol Apple II:KBD_NOTE_P1
- added KBDN? (x3): 3, symbol Apple II:TPK_TRIANGLE_NOTE
- added KBDN?: 1, symbol Apple II:KBD_NOTE_J1_2PIN
- added KBDN?: 8, symbol Apple II:TPK_TRIANGLE_NOTE
- added KBDN?: 19, symbol Apple II:KBD_NOTE_P1
- added KBDN?: 20, symbol Apple II:KBD_NOTE_P1
- added N?: 25µS, symbol Apple II:SINE_WAVE
- added N?: SINE_WAVE, symbol Apple II:SINE_WAVE
- added R1: 51K, symbol Device:R_US
- added R10, R5: 3K, symbol Device:R_US
- added R2, R3, R6: 4.7K, symbol Device:R_US
- added R4: 220Ω, symbol Device:R_US
- added R7: 220K, symbol Device:R_US
- added R8: 510K, symbol Device:R_US
- added S1: KEY 56, symbol Switch:SW_SPDT
- added S?: TPK_S2, symbol Apple II:TPK_S2
- added SW13: RESET (13), symbol Switch:SW_SPST
- added SW25: RPT (25), symbol Switch:SW_SPST
- added SW28: CONTROL (28), symbol Switch:SW_SPST
- added SW42: L.H. SHIFT (42), symbol Switch:SW_SPST
- added SW53: R.H. SHIFT (53), symbol Switch:SW_SPST
- added U? (x4): TPK_B3_7400, symbol Apple II:TPK_B3_7400
- added U?: TPK_B6_AY-5-3600-931, symbol Apple II:TPK_B6_AY-5-3600-931
- added U? (x2): TPK_B4_74LS00, symbol Apple II:TPK_B4_74LS00
- added U?: TPK_NUMERIC_PAD, symbol Apple II:TPK_NUMERIC_PAD
- added U?: TPK_B5_74LS04, symbol Apple II:TPK_B5_74LS04
- added U?: TPK_B2_555, Package_SO:SOIC-8_3.9x4.9mm_P1.27mm, symbol Apple II:TPK_B2_555
Connections:
- new net: KBDN2., U?.3
- new net: R6.1, U?., U?.1
- new net: U?.2, U?.6
- new net: KBDN5., U?.2
- new net: KBDN24., SW42.1 (A), SW53.1 (A)
- new net: KBDN23., SW42.2 (B), SW53.2 (B)
- new net: C5.1, U?.1
- new net: U?.11 (B4), U?.9
- new net: U?.12 (B3), U?.5
- new net: U?.11, U?.13 (B2)
- new net: U?.13, U?.14 (B1)
- new net: KBDN5., U?.17 (Y0)
- new net: KBDN6., U?.18 (Y1)
- new net: KBDN7., U?.19 (Y2)
- new net: C5.2, R1.1, U?.2
- new net: KBDN8., U?.20 (Y3)
- new net: KBDN9., U?.21 (Y4)
- new net: KBDN10., U?.22 (Y5)
- new net: C4.1, KBDN15., U?.27 (V_{GG})
- new net: U?.11, U?.28 (CONTROL)
- new net: U?.29 (SHIFT), U?.8
- new net: R1.2, U?.3
- new net: KBDN2., U?.36 (X4)
- new net: KBDN11., U?.37 (X3)
- new net: KBDN13., U?.38 (X2)
- new net: KBDN14., U?.39 (X1)
- new net: KBDN?., U?.4 (AKO)
- new net: KBDN17., U?.40 (X0)
- new net: U?.1, U?.2, U?.8 (B7)
- new net: R4.1, R6.2, U?.
- new net: C6.1, R4.2, R5.2
- new net: KBDN24., R2.1, U?.10, U?.9
- new net: D?., KBDN23.
- new net: D?., KBDN4.
- new net: KBDN7., U?.3
- new net: KBDN21., R3.2, S1.1 (A), U?.12, U?.13
- new net: KBDN21., SW13.2 (B)
- new net: KBD?.X1, KBDN14.
- new net: KBD?.Y1, KBDN6.
- new net: C8.2, KBDN?., R10.1, U?.4 (~{R})
- new net: KBD?.X2, KBDN13.
- new net: KBD?.X3, KBDN11.
- new net: KBD?.X0, KBDN17.
- new net: KBDN13., U?.10
- new net: KBDN12., U?.12
- new net: KBDN6., U?.4
- new net: KBDN10., U?.6
- new net: KBDN11., U?.8
- new net: KBDN23., SW28.1 (A)
- new net: KBDN3., SW28.2 (B)
- new net: C7.2, R7.1, U?.2 (TR), U?.6 (TH)
- new net: R7.2, R8.2, U?.7 (DIS)
- new net: KBDN3., S1.2 (B)
- new net: KBD?.Y0, KBDN5.
- new net: C6.2, U?.3 (OUT)
- new net: KBD?.X4, KBDN2.
- new net: KBDN?., SW25.1 (A)
- new net: KBDN?., SW25.2 (B)
- new net: KBD?.Y3, KBDN8.
- new net: KBD?.Y2, KBDN7.
- new net: KBD?.Y4, KBDN9.
- new net: KBD?.Y5, KBDN10.
- new net: KBDN56., S1.3 (C)
- new net: KBDN22., KBDN3.
- new net: KBDN22., SW13.1 (A)
- new net +5V: C1.1, C3.2, KBDN4., KBDN?., R2.2, R3.1, R5.1, R8.1, U?.30 (V_{CC}), U?.8 (VCC)
- new net -12V: KBDN15.
- new net ASR OPTION: S?., U?.1, U?.10 (ASR_OPTION_B5), U?.3, U?.9 (ASR_OPTION_B6)
- new net B1: KBDN12.
- new net B2: KBDN13.
- new net B3: KBDN10.
- new net B4: KBDN11.
- new net B5: KBDN6.
- new net B6: KBDN5.
- new net B7: KBDN7.
- new net DATA STROBE OUTPUT: U?.16 (DATA_STROBE_OUTPUT), U?.4, U?.5
- new net Earth: C1.2, C2.2, C3.1, C4.2, C7.1, C8.1, KBDN23., KBDN23., KBDN23., KBDN56., KBDN8., R10.2, U?.1 (GND), U?.15 (V_{DD})
- new net GND: KBDN8.
- new net STROBE DELAY (8MS): C2.1, U?.31 (STROBE_DELAY)
- new net UPPER/LOWER OPTION: S?., U?.6 (UPPER/LOWER_OPTION_B9), U?.7 (UPPER/LOWER_OPTION_B8)
- new net X5: U?.35 (X5), U?.4 (X5)
- new net X6: U?.34 (X6), U?.5 (X6)
- new net X7: U?.33 (X7), U?.9 (X7)
- new net X8: U?.32 (X8), U?.8 (X8)
- new net Y6: KBD?.Y6, KBDN12., U?.2 (Y6), U?.23 (Y6)
- new net Y7: KBD?.Y7, KBDN15., U?.1 (Y7), U?.24 (Y7)
- new net Y8: KBD?.Y8, KBDN16., U?.25 (Y8), U?.6 (Y8)
- new net Y9: KBD?.Y9, KBDN18., U?.26 (Y9), U?.7 (Y9)
Other:
- note added: "(LSB)"
- note added: "OUTPUT DATA (DATA TRUE = HIGH)"
- note added: "STROBE"
- note added: "TO AY- 5-3600- 931 MATRIX"
- title: (none) -> Apple II - Two Piece Keyboard

Commit message: Working on Apple II - Sheet 23
My eyes said I need a break :smile:
Parts:
- added N?: TPK_NOTES, symbol Apple II:TPK_NOTES
Connections:
- net at D?.: now also KBDN4.; no longer KBDN23.
- new net: D?., KBDN23.
Changed lines of the file:
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@@
     (pin "2")
+  )
+  (symbol (lib_id "Apple II:TPK_NOTES") (at 353.06 207.01 0) (unit 1)
+    (in_bom yes) (on_board yes) (fields_autoplaced)
+    (property "Reference" "N?" (id 0) (at 328.93 194.31 0)
+      (effects (font (size 1.27 1.27)) hide)
+    )
+    (property "Value" "TPK_NOTES" (id 1) (at 328.93 191.77 0)
+      (effects (font (size 1.27 1.27)) hide)
+    )
+    (property "Footprint" "" (id 2) (at 328.93 194.31 0)
+      (effects (font (size 1.27 1.27)) hide)
+    )
+    (property "Datasheet" "" (id 3) (at 328.93 194.31 0)
+      (effects (font (size 1.27 1.27)) hide)
+    )
   )
   (symbol (lib_id "Apple II:TPK_B6_AY-5-3600-931") (at 148.59 80.01 0) (unit 1)

Commit message: Working on the Apple II Sheet 23
Connections:
- net at D?.: now also KBDN4.; no longer KBDN23.
- new net: D?., KBDN23.

Commit message: More Apple II Power Supply work
Connections:
- net at D?.: now also KBDN4.; no longer KBDN23.
- new net: D?., KBDN23.

Commit message: Apple II Complete!
All done!  Release to follow!
Connections:
- net at D?.: now also KBDN4.; no longer KBDN23.
- new net: D?., KBDN23.
