File: NABU/untitled.kicad_sch (KiCad schematic)
At the start: 0 parts

Commit message: Finished NABU Page 1
Other:
- company: NABU Network Corporation -> (none)
- title: NABU PC Schematic Cover Sheet -> (none)
Changed lines of the file:
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@@
 (kicad_sch (version 20211123) (generator eeschema)
-  (paper "A0")
-  (title_block
-    (title "NABU PC Schematic Cover Sheet")
-    (date "2022-12-21")
-    (rev "11/16/89")
-    (company "NABU Network Corporation")
-    (comment 1 "Original Schematic by Unknown")
-    (comment 2 "https://github.com/omega9380/Retro-Schematics")
-    (comment 3 "Replication by Omega9380 - December 2022")
-    (comment 4 "Source: NABU Consolidated Documentation v1.0a.pdf by starkscon")
-  )
+  (paper "A4")
 )
